File: base.sch (EAGLE design)
At the start: 20 parts

Commit message: no message
Parts:
- removed 5V-DIP(PWR), 5V-IR(DIG), 5V-LED(DIG), 5V-SEN(PWR), GND(DIG), GND-SEN(PWR), SEN-SIGNAL(ANA): (no value), pinhead:PINHD-1X1
- removed DIP-PINS: (no value), pinhead:PINHD-1X5
- removed X1: (no value), con-molex:KK-156-4
- added J1: (no value), SparkFun-Connectors:CONN_07
- added J2: 455-1750-1-ND, SparkFun-Connectors:CONN_03
- added J3, J4: (no value), SparkFun-Connectors:CONN_01
- added U$4: DF1BZ-4DP-2.5DSA, ferraris_sensor_project:DF1BZ-4DP-2.5DSA
- R1: value 10kOhm -> 10 kOhm
- R2: value 5kOhm -> 100 Ohm
- R3: value 100Ohm -> 39 Ohm
- R4: value 220Ohm -> 82 Ohm
- R5, R6, R7, R8, R9: value 680kOhm -> 680 kOhm
Connections:
- removed net N$10: 5V-DIP(PWR).1, ID-DIP.1, ID-DIP.2, ID-DIP.3, ID-DIP.4, ID-DIP.5
- removed net N$11: DIP-PINS.1, ID-DIP.10, R9.1
- removed net N$12: DIP-PINS.2, ID-DIP.9, R8.1
- removed net N$13: DIP-PINS.3, ID-DIP.8, R7.1
- removed net N$14: DIP-PINS.4, ID-DIP.7, R6.1
- removed net N$15: DIP-PINS.5, ID-DIP.6, R5.1
- removed net N$16: GND(DIG).1, LED1.C, R5.2, R6.2, R7.2, R8.2, R9.2, X1-2.S
- removed net N$4: R3.2, X1-1.S
- removed net N$5: 5V-IR(DIG).1, R3.1
- removed net N$6: 5V-LED(DIG).1, R4.1
- removed net N$8: GND-SEN(PWR).1, X1-4.S
- removed net N$9: 5V-SEN(PWR).1, R2.2
- new net DIP_1: ID-DIP.10, J1.6, R9.1
- new net DIP_2: ID-DIP.9, J1.5, R8.1
- new net DIP_3: ID-DIP.8, J1.1, R7.1
- new net DIP_4: ID-DIP.7, J2.3, R6.1
- new net DIP_5: ID-DIP.6, J2.1, R5.1
- new net DIP_PWR: ID-DIP.1, ID-DIP.2, ID-DIP.3, ID-DIP.4, ID-DIP.5, J2.2
- new net GND_A: J3.1, U$4.4
- new net GND_D: J1.7, LED1.C, R5.2, R6.2, R7.2, R8.2, R9.2, U$4.2
- new net IR_PWR: J1.3, R3.1
- new net LED_PWR: J1.4, R4.1
- new net SIG: J4.1, R1.3, U$4.3
- new net TR_PWR: J1.2, R2.2
- net N$2: now also R3.2, U$4.1; no longer R1.3, SEN-SIGNAL(ANA).1, X1-3.S
Other:
- note removed: "A"
- note removed: "CATH"
- note removed: "COLL"
- note removed: "E"
- moved on the sheet: ID-DIP, LED1, R1, R2, R3, R4, R5, R6, R7, R8, R9

Commit message: no message
Parts:
- removed ID-DIP: SWS005, smd-special:SWS005
- removed R1: 10 kOhm, rcl:POTENTIOMETER_PT-10
- added U$2: DIP-SW-CTS-208-5, ferraris_sensor_project:DIP-SW-CTS-208-5
- added U$3: 93PR10KLF, ferraris_sensor_project:93PR10KLF
- J2: value 455-1750-1-ND -> (none)
- LED1: device led:LED3MM -> SparkFun-LED:LED-3MM-NO_SILK
- R2: value 100 Ohm -> 100; device rcl:R-EU_0204/5 -> rcl:R-EU_0204/7
- R3: value 39 Ohm -> 39; device rcl:R-EU_0204/5 -> rcl:R-EU_0204/7
- R4: value 82 Ohm -> 82; device rcl:R-EU_0204/5 -> rcl:R-EU_0204/7
- R5, R6, R7, R8, R9: value 680 kOhm -> 680k; device resistor:R-EU_0204/5 -> rcl:R-EU_0204/7
- renumbered U$4 to U$1
Connections:
- net DIP_1: now also U$2.1_ON; no longer ID-DIP.10
- net DIP_2: now also U$2.2_ON; no longer ID-DIP.9
- net DIP_3: now also U$2.3_ON; no longer ID-DIP.8
- net DIP_4: now also U$2.4_ON; no longer ID-DIP.7
- net DIP_5: now also U$2.5_ON; no longer ID-DIP.6
- net DIP_PWR: now also U$2.1_OFF, U$2.2_OFF, U$2.3_OFF, U$2.4_OFF, U$2.5_OFF; no longer ID-DIP.1, ID-DIP.2, ID-DIP.3, ID-DIP.4, ID-DIP.5
- net GND_A: now also R2.2; no longer U$1.4
- net N$1: now also U$3.P$2; no longer R1.2
- net SIG: now also U$3.P$3; no longer R1.3
- net TR_PWR: now also U$1.4; no longer R2.2
Other:
- moved on the sheet: R2

Commit message: no message
Parts:
- R2.100: value 100 -> (none)
- R3.39: value 39 -> (none)
- R4.82: value 82 -> (none)
- R5.680K, R6.680K, R7.680K, R8.680K, R9.680K: value 680k -> (none)
- renumbered LED1 to LED, R2 to R2.100, R3 to R3.39, R4 to R4.82, R5 to R5.680K, R6 to R6.680K, R7 to R7.680K, R8 to R8.680K, R9 to R9.680K, U$3 to R1.10K
Changed lines of the file:
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@@
 </classes>
 <parts>
-<part name="LED1" library="SparkFun-LED" deviceset="LED" device="-3MM-NO_SILK"/>
-<part name="R2" library="rcl" library_urn="urn:adsk.eagle:library:334" deviceset="R-EU_" device="0204/7" package3d_urn="urn:adsk.eagle:package:23498/1" value="100"/>
-<part name="R3" library="rcl" library_urn="urn:adsk.eagle:library:334" deviceset="R-EU_" device="0204/7" package3d_urn="urn:adsk.eagle:package:23498/1" value="39"/>
-<part name="R4" library="rcl" library_urn="urn:adsk.eagle:library:334" deviceset="R-EU_" device="0204/7" package3d_urn="urn:adsk.eagle:package:23498/1" value="82"/>
-<part name="R5" library="rcl" library_urn="urn:adsk.eagle:library:334" deviceset="R-EU_" device="0204/7" package3d_urn="urn:adsk.eagle:package:23498/1" value="680k"/>
-<part name="R6" library="rcl" library_urn="urn:adsk.eagle:library:334" deviceset="R-EU_" device="0204/7" package3d_urn="urn:adsk.eagle:package:23498/1" value="680k"/>
-<part name="R7" library="rcl" library_urn="urn:adsk.eagle:library:334" deviceset="R-EU_" device="0204/7" package3d_urn="urn:adsk.eagle:package:23498/1" value="680k"/>
-<part name="R8" library="rcl" library_urn="urn:adsk.eagle:library:334" deviceset="R-EU_" device="0204/7" package3d_urn="urn:adsk.eagle:package:23498/1" value="680k"/>
-<part name="R9" library="rcl" library_urn="urn:adsk.eagle:library:334" deviceset="R-EU_" device="0204/7" package3d_urn="urn:adsk.eagle:package:23498/1" value="680k"/>
+<part name="LED" library="SparkFun-LED" deviceset="LED" device="-3MM-NO_SILK"/>
+<part name="R2.100" library="rcl" library_urn="urn:adsk.eagle:library:334" deviceset="R-EU_" device="0204/7" package3d_urn="urn:adsk.eagle:package:23498/1"/>
+<part name="R3.39" library="rcl" library_urn="urn:adsk.eagle:library:334" deviceset="R-EU_" device="0204/7" package3d_urn="urn:adsk.eagle:package:23498/1"/>
+<part name="R4.82" library="rcl" library_urn="urn:adsk.eagle:library:334" deviceset="R-EU_" device="0204/7" package3d_urn="urn:adsk.eagle:package:23498/1"/>
+<part name="R5.680K" library="rcl" library_urn="urn:adsk.eagle:library:334" deviceset="R-EU_" device="0204/7" package3d_urn="urn:adsk.eagle:package:23498/1"/>
+<part name="R6.680K" library="rcl" library_urn="urn:adsk.eagle:library:334" deviceset="R-EU_" device="0204/7" package3d_urn="urn:adsk.eagle:package:23498/1"/>
+<part name="R7.680K" library="rcl" library_urn="urn:adsk.eagle:library:334" deviceset="R-EU_" device="0204/7" package3d_urn="urn:adsk.eagle:package:23498/1"/>
+<part name="R8.680K" library="rcl" library_urn="urn:adsk.eagle:library:334" deviceset="R-EU_" device="0204/7" package3d_urn="urn:adsk.eagle:package:23498/1"/>
+<part name="R9.680K" library="rcl" library_urn="urn:adsk.eagle:library:334" deviceset="R-EU_" device="0204/7" package3d_urn="urn:adsk.eagle:package:23498/1"/>
 <part name="J1" library="SparkFun-Connectors" deviceset="CONN_07" device=""/>
 <part name="J2" library="SparkFun-Connectors" deviceset="CONN_03" device=""/>
@@
 <part name="U$1" library="ferraris_sensor_project" deviceset="DF1BZ-4DP-2.5DSA" device=""/>
 <part name="U$2" library="ferraris_sensor_project" deviceset="DIP-SW-CTS-208-5" device=""/>
-<part name="U$3" library="ferraris_sensor_project" deviceset="93PR10KLF" device=""/>
+<part name="R1.10K" library="ferraris_sensor_project" deviceset="93PR10KLF" device=""/>
 </parts>
 <sheets>
@@
 </plain>
 <instances>
-<instance part="LED1" gate="G$1" x="50.8" y="20.32" rot="R90"/>
-<instance part="R2" gate="G$1" x="58.42" y="43.18"/>
-<instance part="R3" gate="G$1" x="5.08" y="40.64"/>
-<instance part="R4" gate="G$1" x="38.1" y="20.32"/>
-<instance part="R5" gate="G$1" x="33.02" y="7.62" rot="R180"/>
-<instance part="R6" gate="G$1" x="33.02" y="0" rot="R180"/>
-<instance part="R7" gate="G$1" x="33.02" y="-7.62" rot="R180"/>
-<instance part="R8" gate="G$1" x="33.02" y="-15.24" rot="R180"/>
-<instance part="R9" gate="G$1" x="33.02" y="-22.86" rot="R180"/>
+<instance part="LED" gate="G$1" x="50.8" y="20.32" rot="R90"/>
+<instance part="R2.100" gate="G$1" x="58.42" y="43.18"/>
+<instance part="R3.39" gate="G$1" x="5.08" y="40.64"/>
+<instance part="R4.82" gate="G$1" x="38.1" y="20.32"/>
+<instance part="R5.680K" gate="G$1" x="33.02" y="7.62" rot="R180"/>
+<instance part="R6.680K" gate="G$1" x="33.02" y="0" rot="R180"/>
+<instance part="R7.680K" gate="G$1" x="33.02" y="-7.62" rot="R180"/>
+<instance part="R8.680K" gate="G$1" x="33.02" y="-15.24" rot="R180"/>
+<instance part="R9.680K" gate="G$1" x="33.02" y="-22.86" rot="R180"/>
 <instance part="J1" gate="G$1" x="-12.7" y="12.7"/>
 <instance part="J2" gate="J$1" x="-15.24" y="-5.08"/>
@@
 <instance part="U$1" gate="G$1" x="15.24" y="43.18" rot="R90"/>
 <instance part="U$2" gate="G$1" x="55.88" y="-25.4"/>
-<instance part="U$3" gate="G$1" x="35.56" y="43.18"/>
+<instance part="R1.10K" gate="G$1" x="35.56" y="43.18"/>
 </instances>
 <busses>
@@
 <net name="N$3" class="0">
 <segment>
-<pinref part="R4" gate="G$1" pin="2"/>
-<pinref part="LED1" gate="G$1" pin="A"/>
+<pinref part="R4.82" gate="G$1" pin="2"/>
+<pinref part="LED" gate="G$1" pin="A"/>
 <wire x1="43.18" y1="20.32" x2="48.26" y2="20.32" width="0.1524" layer="91"/>
 </segment>
@@
 </segment>
 <segment>
-<pinref part="R5" gate="G$1" pin="2"/>
+<pinref part="R5.680K" gate="G$1" pin="2"/>
 <wire x1="27.94" y1="7.62" x2="22.86" y2="7.62" width="0.1524" layer="91"/>
 <wire x1="22.86" y1="0" x2="22.86" y2="7.62" width="0.1524" layer="91"/>
-<pinref part="R6" gate="G$1" pin="2"/>
+<pinref part="R6.680K" gate="G$1" pin="2"/>
 <wire x1="27.94" y1="0" x2="22.86" y2="0" width="0.1524" layer="91"/>
 <junction x="22.86" y="0"/>
 <wire x1="22.86" y1="-7.62" x2="22.86" y2="0" width="0.1524" layer="91"/>
-<pinref part="R7" gate="G$1" pin="2"/>
+<pinref part="R7.680K" gate="G$1" pin="2"/>
 <wire x1="27.94" y1="-7.62" x2="22.86" y2="-7.62" width="0.1524" layer="91"/>
 <junction x="22.86" y="-7.62"/>
 <wire x1="22.86" y1="-15.24" x2="22.86" y2="-7.62" width="0.1524" layer="91"/>
-<pinref part="R8" gate="G$1" pin="2"/>
+<pinref part="R8.680K" gate="G$1" pin="2"/>
 <wire x1="27.94" y1="-15.24" x2="22.86" y2="-15.24" width="0.1524" layer="91"/>
 <junction x="22.86" y="-15.24"/>
-<pinref part="R9" gate="G$1" pin="2"/>
+<pinref part="R9.680K" gate="G$1" pin="2"/>
 <wire x1="27.94" y1="-22.86" x2="22.86" y2="-22.86" width="0.1524" layer="91"/>
 <wire x1="22.86" y1="-22.86" x2="22.86" y2="-15.24" width="0.1524" layer="91"/>
@@
 </segment>
 <segment>
-<pinref part="LED1" gate="G$1" pin="C"/>
+<pinref part="LED" gate="G$1" pin="C"/>
 <wire x1="55.88" y1="20.32" x2="60.96" y2="20.32" width="0.1524" layer="91"/>
 <label x="60.96" y="20.32" size="1.778" layer="95"/>
@@
 <segment>
 <wire x1="50.8" y1="-15.24" x2="50.8" y2="-12.7" width="0.1524" layer="91"/>
-<pinref part="R9" gate="G$1" pin="1"/>
+<pinref part="R9.680K" gate="G$1" pin="1"/>
 <wire x1="50.8" y1="-12.7" x2="50.8" y2="2.54" width="0.1524" layer="91"/>
 <wire x1="38.1" y1="-22.86" x2="43.18" y2="-22.86" width="0.1524" layer="91"/>
@@
 <segment>
 <wire x1="53.34" y1="-15.24" x2="53.34" y2="-10.16" width="0.1524" layer="91"/>
-<pinref part="R8" gate="G$1" pin="1"/>
+<pinref part="R8.680K" gate="G$1" pin="1"/>
 <wire x1="53.34" y1="-10.16" x2="53.34" y2="2.54" width="0.1524" layer="91"/>
 <wire x1="38.1" y1="-15.24" x2="40.64" y2="-15.24" width="0.1524" layer="91"/>
@@
 </segment>
 <segment>
-<pinref part="R4" gate="G$1" pin="1"/>
+<pinref part="R4.82" gate="G$1" pin="1"/>
 <wire x1="25.4" y1="20.32" x2="33.02" y2="20.32" width="0.1524" layer="91"/>
 <label x="17.78" y="17.78" size="1.778" layer="95"/>
@@
 </segment>
 <segment>
-<pinref part="R3" gate="G$1" pin="1"/>
+<pinref part="R3.39" gate="G$1" pin="1"/>
 <wire x1="-7.62" y1="40.64" x2="0" y2="40.64" width="0.1524" layer="91"/>
 <label x="-12.7" y="38.1" size="1.778" layer="95"/>
@@
 <segment>
 <wire x1="55.88" y1="-15.24" x2="55.88" y2="-7.62" width="0.1524" layer="91"/>
-<pinref part="R7" gate="G$1" pin="1"/>
+<pinref part="R7.680K" gate="G$1" pin="1"/>
 <wire x1="55.88" y1="-7.62" x2="55.88" y2="2.54" width="0.1524" layer="91"/>
 <wire x1="38.1" y1="-7.62" x2="55.88" y2="-7.62" width="0.1524" layer="91"/>
@@
 <segment>
 <wire x1="58.42" y1="-15.24" x2="58.42" y2="-5.08" width="0.1524" layer="91"/>
-<pinref part="R6" gate="G$1" pin="1"/>
+<pinref part="R6.680K" gate="G$1" pin="1"/>
 <wire x1="58.42" y1="-5.08" x2="58.42" y2="2.54" width="0.1524" layer="91"/>
 <wire x1="38.1" y1="0" x2="40.64" y2="0" width="0.1524" layer="91"/>
@@
 <segment>
 <wire x1="60.96" y1="-15.24" x2="60.96" y2="-2.54" width="0.1524" layer="91"/>
-<pinref part="R5" gate="G$1" pin="1"/>
+<pinref part="R5.680K" gate="G$1" pin="1"/>
 <wire x1="60.96" y1="-2.54" x2="60.96" y2="2.54" width="0.1524" layer="91"/>
 <wire x1="38.1" y1="7.62" x2="43.18" y2="7.62" width="0.1524" layer="91"/>
@@
 </segment>
 <segment>
-<pinref part="R2" gate="G$1" pin="2"/>
+<pinref part="R2.100" gate="G$1" pin="2"/>
 <wire x1="63.5" y1="43.18" x2="68.58" y2="43.18" width="0.1524" layer="91"/>
 <label x="68.58" y="43.18" size="1.778" layer="95"/>
@@
 <junction x="30.48" y="35.56"/>
 <pinref part="U$1" gate="G$1" pin="3"/>
-<pinref part="U$3" gate="G$1" pin="P$3"/>
+<pinref part="R1.10K" gate="G$1" pin="P$3"/>
 <wire x1="40.56" y1="37.88" x2="40.56" y2="35.56" width="0.1524" layer="91"/>
 </segment>
@@
 <net name="N$2" class="0">
 <segment>
-<pinref part="R3" gate="G$1" pin="2"/>
+<pinref part="R3.39" gate="G$1" pin="2"/>
 <wire x1="10.16" y1="40.64" x2="12.24" y2="40.64" width="0.1524" layer="91"/>
 <wire x1="12.24" y1="40.64" x2="12.24" y2="43.18" width="0.1524" layer="91"/>
@@
 <net name="N$1" class="0">
 <segment>
-<pinref part="U$3" gate="G$1" pin="P$2"/>
-<pinref part="R2" gate="G$1" pin="1"/>
+<pinref part="R1.10K" gate="G$1" pin="P$2"/>
+<pinref part="R2.100" gate="G$1" pin="1"/>
 <wire x1="50.66" y1="45.78" x2="50.66" y2="43.18" width="0.1524" layer="91"/>
 <wire x1="50.66" y1="43.18" x2="53.34" y2="43.18" width="0.1524" layer="91"/>

Commit message: no message
Connections:
- net DIP_3: now also J2.1; no longer J1.1
- net DIP_5: now also J1.1; no longer J2.1
- net DIP_PWR: now also J1.3; no longer J2.2
- net IR_PWR: now also J2.2; no longer J1.3
Changed lines of the file:
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@@
 <?xml version="1.0" encoding="utf-8"?>
 <!DOCTYPE eagle SYSTEM "eagle.dtd">
-<eagle version="8.7.0">
+<eagle version="8.7.1">
 <drawing>
 <settings>
@@
 <net name="IR_PWR" class="0">
 <segment>
-<pinref part="J1" gate="G$1" pin="3"/>
-<wire x1="-7.62" y1="12.7" x2="-5.08" y2="12.7" width="0.1524" layer="91"/>
-<label x="-5.08" y="12.7" size="1.778" layer="95"/>
-</segment>
-<segment>
 <pinref part="R3.39" gate="G$1" pin="1"/>
 <wire x1="-7.62" y1="40.64" x2="0" y2="40.64" width="0.1524" layer="91"/>
 <label x="-12.7" y="38.1" size="1.778" layer="95"/>
+</segment>
+<segment>
+<pinref part="J2" gate="J$1" pin="2"/>
+<wire x1="-7.62" y1="-5.08" x2="-5.08" y2="-5.08" width="0.1524" layer="91"/>
+<label x="-5.08" y="-5.08" size="1.778" layer="95"/>
 </segment>
 </net>
@@
 </net>
 <net name="DIP_3" class="0">
-<segment>
-<pinref part="J1" gate="G$1" pin="1"/>
-<wire x1="-7.62" y1="7.62" x2="-5.08" y2="7.62" width="0.1524" layer="91"/>
-<label x="-5.08" y="7.62" size="1.778" layer="95"/>
-</segment>
 <segment>
 <wire x1="55.88" y1="-15.24" x2="55.88" y2="-7.62" width="0.1524" layer="91"/>
@@
 <wire x1="56.34" y1="-20.86" x2="56.34" y2="-15.24" width="0.1524" layer="91"/>
 <wire x1="56.34" y1="-15.24" x2="55.88" y2="-15.24" width="0.1524" layer="91"/>
+</segment>
+<segment>
+<pinref part="J2" gate="J$1" pin="1"/>
+<wire x1="-7.62" y1="-7.62" x2="-5.08" y2="-7.62" width="0.1524" layer="91"/>
+<label x="-5.08" y="-7.62" size="1.778" layer="95"/>
 </segment>
 </net>
@@
 </net>
 <net name="DIP_PWR" class="0">
-<segment>
-<pinref part="J2" gate="J$1" pin="2"/>
-<wire x1="-7.62" y1="-5.08" x2="-5.08" y2="-5.08" width="0.1524" layer="91"/>
-<label x="-5.08" y="-5.08" size="1.778" layer="95"/>
-</segment>
 <segment>
 <wire x1="60.96" y1="-38.1" x2="58.42" y2="-38.1" width="0.1524" layer="91"/>
@@
 <wire x1="60.34" y1="-35.56" x2="60.96" y2="-35.56" width="0.1524" layer="91"/>
 </segment>
+<segment>
+<pinref part="J1" gate="G$1" pin="3"/>
+<wire x1="-7.62" y1="12.7" x2="-5.08" y2="12.7" width="0.1524" layer="91"/>
+<label x="-5.08" y="12.7" size="1.778" layer="95"/>
+</segment>
 </net>
 <net name="DIP_5" class="0">
-<segment>
-<pinref part="J2" gate="J$1" pin="1"/>
-<wire x1="-7.62" y1="-7.62" x2="-5.08" y2="-7.62" width="0.1524" layer="91"/>
-<label x="-5.08" y="-7.62" size="1.778" layer="95"/>
-</segment>
 <segment>
 <wire x1="60.96" y1="-15.24" x2="60.96" y2="-2.54" width="0.1524" layer="91"/>
@@
 <wire x1="60.34" y1="-15.24" x2="60.96" y2="-15.24" width="0.1524" layer="91"/>
 </segment>
-</net>
+<segment>
+<pinref part="J1" gate="G$1" pin="1"/>
+<wire x1="-7.62" y1="7.62" x2="-5.08" y2="7.62" width="0.1524" layer="91"/>
+<label x="-5.08" y="7.62" size="1.778" layer="95"/>
+</segment>
+</net>

Commit message: no message
Connections:
- net DIP_PWR: now also J1.2; no longer J1.3
- net TR_PWR: now also J1.3; no longer J1.2
Changed lines of the file:
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@@
 <net name="TR_PWR" class="0">
-<segment>
-<pinref part="J1" gate="G$1" pin="2"/>
-<wire x1="-7.62" y1="10.16" x2="-5.08" y2="10.16" width="0.1524" layer="91"/>
-<label x="-5.08" y="10.16" size="1.778" layer="95"/>
-</segment>
 <segment>
 <wire x1="21.24" y1="43.18" x2="21.24" y2="40.64" width="0.1524" layer="91"/>
@@
 <label x="20.32" y="38.1" size="1.778" layer="95"/>
 <pinref part="U$1" gate="G$1" pin="4"/>
+</segment>
+<segment>
+<pinref part="J1" gate="G$1" pin="3"/>
+<wire x1="-7.62" y1="12.7" x2="-5.08" y2="12.7" width="0.1524" layer="91"/>
+<label x="-5.08" y="12.7" size="1.778" layer="95"/>
 </segment>
 </net>
@@
 </segment>
 <segment>
-<pinref part="J1" gate="G$1" pin="3"/>
-<wire x1="-7.62" y1="12.7" x2="-5.08" y2="12.7" width="0.1524" layer="91"/>
-<label x="-5.08" y="12.7" size="1.778" layer="95"/>
+<pinref part="J1" gate="G$1" pin="2"/>
+<wire x1="-7.62" y1="10.16" x2="-5.08" y2="10.16" width="0.1524" layer="91"/>
+<label x="-5.08" y="10.16" size="1.778" layer="95"/>
 </segment>
 </net>

Commit message: updated layout and part
Parts:
- removed R1.10K: 93PR10KLF, ferraris_sensor_project:93PR10KLF
- added U$3: CT6EP103, ferraris_sensor_project:CT6EP103
Connections:
- net N$1: now also U$3.P$3; no longer R1.10K.P$2
- net SIG: now also U$3.P$2; no longer R1.10K.P$3
Changed lines of the file:
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@@
 <part name="U$1" library="ferraris_sensor_project" deviceset="DF1BZ-4DP-2.5DSA" device=""/>
 <part name="U$2" library="ferraris_sensor_project" deviceset="DIP-SW-CTS-208-5" device=""/>
-<part name="R1.10K" library="ferraris_sensor_project" deviceset="93PR10KLF" device=""/>
+<part name="U$3" library="ferraris_sensor_project" deviceset="CT6EP103" device=""/>
 </parts>
 <sheets>
@@
 <instance part="U$1" gate="G$1" x="15.24" y="43.18" rot="R90"/>
 <instance part="U$2" gate="G$1" x="55.88" y="-25.4"/>
-<instance part="R1.10K" gate="G$1" x="35.56" y="43.18"/>
+<instance part="U$3" gate="G$1" x="35.56" y="43.18"/>
 </instances>
 <busses>
@@
 <junction x="30.48" y="35.56"/>
 <pinref part="U$1" gate="G$1" pin="3"/>
-<pinref part="R1.10K" gate="G$1" pin="P$3"/>
 <wire x1="40.56" y1="37.88" x2="40.56" y2="35.56" width="0.1524" layer="91"/>
+<pinref part="U$3" gate="G$1" pin="P$2"/>
 </segment>
 </net>
@@
 <net name="N$1" class="0">
 <segment>
-<pinref part="R1.10K" gate="G$1" pin="P$2"/>
 <pinref part="R2.100" gate="G$1" pin="1"/>
 <wire x1="50.66" y1="45.78" x2="50.66" y2="43.18" width="0.1524" layer="91"/>
 <wire x1="50.66" y1="43.18" x2="53.34" y2="43.18" width="0.1524" layer="91"/>
-</segment>
-</net>
+<pinref part="U$3" gate="G$1" pin="P$3"/>
+</segment>
+</net>

Commit message: fixed
Connections:
- net SIG: now also U$1.4; no longer U$1.3
- net TR_PWR: now also U$1.3; no longer U$1.4
Changed lines of the file:
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@@
 <instance part="X21" gate="G$1" x="30.48" y="30.48"/>
 <instance part="X22" gate="G$1" x="68.58" y="43.18"/>
-<instance part="X23" gate="G$1" x="22.86" y="40.64"/>
+<instance part="X23" gate="G$1" x="22.86" y="27.94"/>
 <instance part="X24" gate="G$1" x="25.4" y="20.32"/>
 <instance part="X25" gate="G$1" x="60.96" y="20.32"/>
@@
 <segment>
 <wire x1="15.24" y1="43.18" x2="15.24" y2="30.48" width="0.1524" layer="91"/>
-<label x="15.24" y="30.48" size="1.778" layer="95"/>
+<label x="5.08" y="30.48" size="1.778" layer="95"/>
 <pinref part="U$1" gate="G$1" pin="2"/>
 </segment>
@@
 <net name="TR_PWR" class="0">
 <segment>
-<wire x1="21.24" y1="43.18" x2="21.24" y2="40.64" width="0.1524" layer="91"/>
-<wire x1="21.24" y1="40.64" x2="22.86" y2="40.64" width="0.1524" layer="91"/>
-<label x="20.32" y="38.1" size="1.778" layer="95"/>
-<pinref part="U$1" gate="G$1" pin="4"/>
-</segment>
-<segment>
 <pinref part="J1" gate="G$1" pin="3"/>
 <wire x1="-7.62" y1="12.7" x2="-5.08" y2="12.7" width="0.1524" layer="91"/>
 <label x="-5.08" y="12.7" size="1.778" layer="95"/>
+</segment>
+<segment>
+<wire x1="21.24" y1="27.94" x2="22.86" y2="27.94" width="0.1524" layer="91"/>
+<label x="22.86" y="25.4" size="1.778" layer="95"/>
+<pinref part="U$1" gate="G$1" pin="3"/>
+<wire x1="18.24" y1="43.18" x2="18.24" y2="27.94" width="0.1524" layer="91"/>
+<wire x1="18.24" y1="27.94" x2="21.24" y2="27.94" width="0.1524" layer="91"/>
 </segment>
 </net>
@@
 <wire x1="30.48" y1="30.48" x2="30.48" y2="35.56" width="0.1524" layer="91"/>
 <label x="30.48" y="30.48" size="1.778" layer="95"/>
-<wire x1="18.24" y1="43.18" x2="18.24" y2="35.56" width="0.1524" layer="91"/>
-<wire x1="18.24" y1="35.56" x2="30.48" y2="35.56" width="0.1524" layer="91"/>
-<junction x="30.48" y="35.56"/>
-<pinref part="U$1" gate="G$1" pin="3"/>
 <wire x1="40.56" y1="37.88" x2="40.56" y2="35.56" width="0.1524" layer="91"/>
 <pinref part="U$3" gate="G$1" pin="P$2"/>
-</segment>
-</net>
+<pinref part="U$1" gate="G$1" pin="4"/>
+<wire x1="21.24" y1="43.18" x2="21.24" y2="35.56" width="0.1524" layer="91"/>
+<wire x1="21.24" y1="35.56" x2="30.48" y2="35.56" width="0.1524" layer="91"/>
+<junction x="30.48" y="35.56"/>
+</segment>
+</net>
