File: dual_sensor.sch (EAGLE design)
At the start: 4 parts

Commit message: no message
Parts:
- added J1: (no value), SparkFun-Connectors:CONN_01
Connections:
- removed net GND2: U$2.GND(PWR)
- net GND: now also R2.1
- net N$3: now also J1.1, R2.2, U$2.GND(PWR); no longer R2.1, U$1.5V(PWR)
- net VCC: now also U$1.5V(PWR); no longer R2.2
Other:
- moved on the sheet: R2
Changed lines of the file:
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@@
 <layer number="230" name="230bmp" color="7" fill="1" visible="yes" active="yes"/>
 <layer number="231" name="231bmp" color="7" fill="1" visible="yes" active="yes"/>
+<layer number="232" name="Eagle3D_PG2" color="7" fill="1" visible="yes" active="yes"/>
+<layer number="233" name="Eagle3D_PG3" color="7" fill="1" visible="yes" active="yes"/>
 <layer number="248" name="Housing" color="7" fill="1" visible="yes" active="yes"/>
 <layer number="249" name="Edge" color="7" fill="1" visible="yes" active="yes"/>
@@
 <part name="GND2" library="SparkFun-PowerSymbols" deviceset="GND" device=""/>
 <part name="SUPPLY1" library="SparkFun-PowerSymbols" deviceset="VCC" device=""/>
+<part name="J1" library="SparkFun-Connectors" deviceset="CONN_01" device=""/>
 </parts>
 <sheets>
@@
 <instance part="U$2" gate="G$1" x="81.28" y="58.42" rot="R180"/>
 <instance part="R1" gate="G$1" x="33.02" y="73.66"/>
-<instance part="R2" gate="G$1" x="73.66" y="27.94"/>
-<instance part="GND1" gate="1" x="50.8" y="38.1"/>
-<instance part="GND2" gate="1" x="76.2" y="45.72"/>
-<instance part="SUPPLY1" gate="G$1" x="83.82" y="27.94"/>
+<instance part="R2" gate="G$1" x="76.2" y="45.72" rot="R180"/>
+<instance part="GND1" gate="1" x="50.8" y="33.02"/>
+<instance part="GND2" gate="1" x="83.82" y="43.18"/>
+<instance part="SUPPLY1" gate="G$1" x="60.96" y="48.26" rot="R90"/>
+<instance part="J1" gate="G$1" x="83.82" y="50.8" rot="R180"/>
 </instances>
 <busses>
@@
 <pinref part="U$1" gate="G$1" pin="GND(DIG)"/>
 <wire x1="54.46" y1="56.92" x2="50.8" y2="56.92" width="0.1524" layer="91"/>
-<wire x1="50.8" y1="56.92" x2="50.8" y2="40.64" width="0.1524" layer="91"/>
+<wire x1="50.8" y1="56.92" x2="50.8" y2="35.56" width="0.1524" layer="91"/>
 <pinref part="GND1" gate="1" pin="GND"/>
+<wire x1="87.78" y1="35.56" x2="86.36" y2="35.56" width="0.1524" layer="91"/>
+<junction x="50.8" y="35.56"/>
 <pinref part="U$2" gate="G$1" pin="GND(DIG)"/>
-<wire x1="87.78" y1="59.92" x2="87.78" y2="40.64" width="0.1524" layer="91"/>
-<wire x1="87.78" y1="40.64" x2="50.8" y2="40.64" width="0.1524" layer="91"/>
-<junction x="50.8" y="40.64"/>
+<wire x1="86.36" y1="35.56" x2="50.8" y2="35.56" width="0.1524" layer="91"/>
+<wire x1="87.78" y1="59.92" x2="91.44" y2="59.92" width="0.1524" layer="91"/>
+<wire x1="91.44" y1="59.92" x2="91.44" y2="35.56" width="0.1524" layer="91"/>
+<wire x1="91.44" y1="35.56" x2="87.78" y2="35.56" width="0.1524" layer="91"/>
+</segment>
+<segment>
+<pinref part="GND2" gate="1" pin="GND"/>
+<pinref part="R2" gate="G$1" pin="1"/>
+<wire x1="81.28" y1="45.72" x2="83.82" y2="45.72" width="0.1524" layer="91"/>
 </segment>
 </net>
@@
 <net name="N$3" class="0">
 <segment>
-<pinref part="U$1" gate="G$1" pin="5V(PWR)"/>
-<pinref part="R2" gate="G$1" pin="1"/>
-<wire x1="67.46" y1="56.92" x2="67.46" y2="27.94" width="0.1524" layer="91"/>
-<wire x1="67.46" y1="27.94" x2="68.58" y2="27.94" width="0.1524" layer="91"/>
+<pinref part="R2" gate="G$1" pin="2"/>
+<wire x1="71.12" y1="45.72" x2="71.12" y2="50.8" width="0.1524" layer="91"/>
+<pinref part="U$2" gate="G$1" pin="GND(PWR)"/>
+<wire x1="71.12" y1="50.8" x2="71.12" y2="56.92" width="0.1524" layer="91"/>
+<wire x1="71.12" y1="56.92" x2="74.78" y2="56.92" width="0.1524" layer="91"/>
+<pinref part="J1" gate="G$1" pin="1"/>
+<wire x1="76.2" y1="50.8" x2="71.12" y2="50.8" width="0.1524" layer="91"/>
+<junction x="71.12" y="50.8"/>
 </segment>
 </net>
 <net name="VCC" class="0">
 <segment>
-<pinref part="R2" gate="G$1" pin="2"/>
+<pinref part="U$1" gate="G$1" pin="5V(PWR)"/>
+<wire x1="67.46" y1="56.92" x2="67.46" y2="48.26" width="0.1524" layer="91"/>
 <pinref part="SUPPLY1" gate="G$1" pin="VCC"/>
-<wire x1="78.74" y1="27.94" x2="83.82" y2="27.94" width="0.1524" layer="91"/>
+<wire x1="60.96" y1="48.26" x2="67.46" y2="48.26" width="0.1524" layer="91"/>
 </segment>
 </net>
-<net name="GND2" class="0">
-<segment>
-<pinref part="U$2" gate="G$1" pin="GND(PWR)"/>
-<pinref part="GND2" gate="1" pin="GND"/>
-<wire x1="74.78" y1="56.92" x2="74.78" y2="48.26" width="0.1524" layer="91"/>
-<wire x1="74.78" y1="48.26" x2="76.2" y2="48.26" width="0.1524" layer="91"/>
-<label x="76.2" y="48.26" size="1.778" layer="95"/>
-</segment>
-</net>
