File: base.brd (EAGLE design)
At the start: 100 x 80 mm, 20 parts

Commit message: no message
Parts:
- removed 5V-DIP(PWR), 5V-IR(DIG), 5V-LED(DIG), 5V-SEN(PWR), GND(DIG), GND-SEN(PWR), SEN-SIGNAL(ANA): (no value), pinhead:1X01
- removed DIP-PINS: (no value), pinhead:1X05
- removed X1: (no value), con-molex:KK-156-4
- added J1: (no value), SparkFun-Connectors:1X07
- added J2: 455-1750-1-ND, SparkFun-Connectors:1X03
- added J3, J4: (no value), SparkFun-Connectors:1X01
- added U$4: DF1BZ-4DP-2.5DSA, ferraris_sensor_project:DF1BZ-4DP-2.5DSA
- R1: value 10kOhm -> 10 kOhm
- R2: value 5kOhm -> 100 Ohm
- R3: value 100Ohm -> 39 Ohm
- R4: value 220Ohm -> 82 Ohm
- R5, R6, R7, R8, R9: value 680kOhm -> 680 kOhm
- moved R2 45.4 mm to (54.6, 55.9), turned to 270 degrees
- moved ID-DIP 31.8 mm to (49.5, 44.5)
- moved R1 31.8 mm to (61.0, 52.1)
- moved R9 30.6 mm to (48.3, 36.8)
- moved R3 27.3 mm to (41.9, 52.1), turned to 90 degrees
- moved R4 21.6 mm to (35.6, 50.8)
- moved R8 20.5 mm to (40.6, 36.8)
- moved R7 12.8 mm to (31.8, 36.8)
- moved LED1 12.7 mm to (36.8, 55.9), turned to 180 degrees
- moved R5 8.13 mm to (31.8, 45.7)
- moved R6 5.39 mm to (31.8, 41.9)
Connections:
- removed net N$10: 5V-DIP(PWR).1, ID-DIP.1, ID-DIP.2, ID-DIP.3, ID-DIP.4, ID-DIP.5
- removed net N$11: DIP-PINS.1, ID-DIP.10, R9.1
- removed net N$12: DIP-PINS.2, ID-DIP.9, R8.1
- removed net N$13: DIP-PINS.3, ID-DIP.8, R7.1
- removed net N$14: DIP-PINS.4, ID-DIP.7, R6.1
- removed net N$15: DIP-PINS.5, ID-DIP.6, R5.1
- removed net N$16: GND(DIG).1, LED1.K, R5.2, R6.2, R7.2, R8.2, R9.2, X1.2
- removed net N$4: R3.2, X1.1
- removed net N$5: 5V-IR(DIG).1, R3.1
- removed net N$6: 5V-LED(DIG).1, R4.1
- removed net N$8: GND-SEN(PWR).1, X1.4
- removed net N$9: 5V-SEN(PWR).1, R2.2
- new net DIP_1: ID-DIP.10, J1.6, R9.1
- new net DIP_2: ID-DIP.9, J1.5, R8.1
- new net DIP_3: ID-DIP.8, J1.1, R7.1
- new net DIP_4: ID-DIP.7, J2.3, R6.1
- new net DIP_5: ID-DIP.6, J2.1, R5.1
- new net DIP_PWR: ID-DIP.1, ID-DIP.2, ID-DIP.3, ID-DIP.4, ID-DIP.5, J2.2
- new net GND_A: J3.1, U$4.3
- new net GND_D: J1.7, LED1.K, R5.2, R6.2, R7.2, R8.2, R9.2, U$4.2
- new net IR_PWR: J1.3, R3.1
- new net LED_PWR: J1.4, R4.1
- new net SIG: J4.1, R1.3, U$4.4
- new net TR_PWR: J1.2, R2.2
- net N$2: now also R3.2, U$4.1; no longer R1.3, SEN-SIGNAL(ANA).1, X1.3

Commit message: no message
Parts:
- removed ID-DIP: SWS005, smd-special:SMS-005
- removed R1: 10 kOhm, rcl:PT-10
- removed U$4: DF1BZ-4DP-2.5DSA, ferraris_sensor_project:DF1BZ-4DP-2.5DSA
- added U$1: DF1BZ-4DP-2.5DSA, ferraris_sensor_project:DF1BZ-4DP-2.5DSA
- added U$2: DIP-SW-CTS-208-5, ferraris_sensor_project:DIP-SW-CTS-208-5
- added U$3: 93PR10KLF, ferraris_sensor_project:93PR10KLF
- J2: value 455-1750-1-ND -> (none)
- LED1: device led:LED3MM -> SparkFun-LED:LED_3MM-NS
- R2: value 100 Ohm -> 100; device rcl:0204/5 -> rcl:0204/7
- R3: value 39 Ohm -> 39; device rcl:0204/5 -> rcl:0204/7
- R4: value 82 Ohm -> 82; device rcl:0204/5 -> rcl:0204/7
- R5, R6, R7, R8, R9: value 680 kOhm -> 680k; device resistor:0204/5 -> rcl:0204/7
- moved LED1 35.3 mm to (67.3, 38.1), turned to 0 degrees
- moved R4 27.3 mm to (59.7, 38.1)
- moved J1 15.7 mm to (27.9, 50.8), turned to 270 degrees
- moved R9 11.4 mm to (36.8, 36.8), turned to 180 degrees
- moved R7 9.16 mm to (36.8, 44.5), turned to 180 degrees
- moved R3 8.13 mm to (36.8, 58.4), turned to 0 degrees
- moved R5 8.13 mm to (36.8, 52.1), turned to 180 degrees
- moved R6 8.13 mm to (36.8, 48.3), turned to 180 degrees
- moved R2 8.03 mm to (62.2, 58.4), turned to 0 degrees
- moved J2 6.35 mm to (27.9, 59.7), turned to 270 degrees
- moved R8 5.39 mm to (36.8, 40.6), turned to 180 degrees
- moved J3 3.81 mm to (76.2, 52.1)
- moved J4 3.81 mm to (76.2, 59.7)
Connections:
- new net P$1: U$3.3
- net DIP_1: now also U$2.1_ON; no longer ID-DIP.10
- net DIP_2: now also U$2.2_ON; no longer ID-DIP.9
- net DIP_3: now also U$2.3_ON; no longer ID-DIP.8
- net DIP_4: now also U$2.4_ON; no longer ID-DIP.7
- net DIP_5: now also U$2.5_ON; no longer ID-DIP.6
- net DIP_PWR: now also U$2.1_OFF, U$2.2_OFF, U$2.3_OFF, U$2.4_OFF, U$2.5_OFF; no longer ID-DIP.1, ID-DIP.2, ID-DIP.3, ID-DIP.4, ID-DIP.5
- net GND_A: now also R2.2; no longer U$4.3
- net GND_D: now also U$1.2; no longer U$4.2
- net N$1: now also U$3.1; no longer R1.2
- net N$2: now also U$1.1; no longer U$4.1
- net SIG: now also U$1.4, U$3.2; no longer R1.3, U$4.4
- net TR_PWR: now also U$1.3; no longer R2.2
Routing:
- net GND_D: track 0.00 -> 69.8 mm
- net DIP_PWR: track 0.00 -> 40.0 mm
- net SIG: track 0.00 -> 35.7 mm
- net TR_PWR: track 0.00 -> 31.1 mm
- net LED_PWR: track 0.00 -> 30.0 mm
- net DIP_5: track 0.00 -> 24.3 mm
- net DIP_4: track 0.00 -> 20.2 mm
- net DIP_3: track 0.00 -> 19.7 mm
- net DIP_1: track 0.00 -> 17.6 mm
- net DIP_2: track 0.00 -> 17.4 mm
- net IR_PWR: track 0.00 -> 14.9 mm
- net N$1: track 0.00 -> 12.8 mm
- net GND_A: track 0.00 -> 12.8 mm
- net N$2: track 0.00 -> 9.08 mm
- net N$3: track 0.00 -> 2.54 mm

Commit message: no message
Parts:
- R2.100: value 100 -> (none)
- R3.39: value 39 -> (none)
- R4.82: value 82 -> (none)
- R5.680K, R6.680K, R7.680K, R8.680K, R9.680K: value 680k -> (none)
- renumbered LED1 to LED, R2 to R2.100, R3 to R3.39, R4 to R4.82, R5 to R5.680K, R6 to R6.680K, R7 to R7.680K, R8 to R8.680K, R9 to R9.680K, U$3 to R1.10K
Routing:
- added copper zone on layer 16, net GND_A
- added copper zone on layer 1, net GND_D
Other:
- board size 100 x 80 mm -> 53.3 x 29.2 mm
- board text added: "SEPL"
- board text added: "v1"

Commit message: no message
Routing:
- net GND_D: track 69.8 -> 0.00 mm
- net DIP_PWR: track 40.0 -> 53.8 mm
- net GND_A: track 12.8 -> 0.00 mm
- net LED_PWR: track 30.0 -> 37.3 mm
- net SIG: track 35.7 -> 41.2 mm
- net IR_PWR: track 14.9 -> 19.2 mm
- net TR_PWR: track 31.1 -> 35.2 mm
- net DIP_5: track 24.3 -> 21.2 mm
- net DIP_1: track 17.6 -> 18.3 mm

Commit message: no message
Parts:
- moved R2.100 1.27 mm to (62.2, 57.1)
Routing:
- net SIG: track 41.2 -> 42.7 mm
- net TR_PWR: track 35.2 -> 36.7 mm
- net N$1: track 12.8 -> 11.5 mm
- net DIP_5: track 21.2 -> 22.4 mm
- net DIP_PWR: track 53.8 -> 54.6 mm

Commit message: no message
Parts:
- moved R9.680K 14.2 mm to (50.8, 39.4), turned to 270 degrees
- moved R5.680K 13.3 mm to (33.0, 39.4), turned to 270 degrees
- moved R8.680K 9.61 mm to (46.4, 39.4), turned to 270 degrees
- moved U$2 8.98 mm to (45.7, 47.0), turned to 180 degrees
- moved R6.680K 8.91 mm to (37.5, 39.4), turned to 270 degrees
- moved R7.680K 7.18 mm to (41.9, 39.4), turned to 270 degrees
- moved R2.100 6.38 mm to (68.6, 56.5)
- moved U$1 5.08 mm to (55.9, 57.1)
- moved R1.10K 1.27 mm to (62.2, 44.5)
- moved LED 0.90 mm to (66.7, 37.5)
- moved R4.82 0.90 mm to (59.1, 37.5)
Routing:
- net SIG: track 42.7 -> 0.00 mm
- net LED_PWR: track 37.3 -> 0.00 mm
- net TR_PWR: track 36.7 -> 0.00 mm
- net DIP_PWR: track 54.6 -> 18.8 mm
- net IR_PWR: track 19.2 -> 0.00 mm
- net DIP_5: track 22.4 -> 4.86 mm
- net DIP_4: track 20.2 -> 4.07 mm
- net DIP_3: track 19.7 -> 4.34 mm
- net DIP_1: track 18.3 -> 33.1 mm
- net N$1: track 11.5 -> 0.00 mm
- net DIP_2: track 17.6 -> 24.6 mm
- net N$2: track 8.92 -> 14.0 mm
- added copper zone on layer 1, net GND_A
- added copper zone on layer 16, net GND_D
- removed copper zone on layer 16, net GND_A
- removed copper zone on layer 1, net GND_D
Other:
- board text removed: "v1"

Commit message: no message
Parts:
- moved LED 38.2 mm to (34.3, 57.8)
- moved R4.82 29.0 mm to (33.0, 50.2), turned to 90 degrees
- moved R2.100 9.53 mm to (61.0, 50.8), turned to 180 degrees
- moved R3.39 8.26 mm to (45.1, 58.4)
- moved R1.10K 5.85 mm to (61.0, 38.7)
- moved U$1 5.12 mm to (61.0, 56.5)
- moved U$2 4.45 mm to (50.2, 47.0)
Connections:
- net DIP_3: now also J2.1; no longer J1.1
- net DIP_5: now also J1.1; no longer J2.1
- net DIP_PWR: now also J1.3; no longer J2.2
- net IR_PWR: now also J2.2; no longer J1.3
Routing:
- net DIP_PWR: track 18.8 -> 53.9 mm
- net TR_PWR: track 0.00 -> 34.7 mm
- net SIG: track 0.00 -> 32.9 mm
- net DIP_3: track 4.34 -> 29.4 mm
- net DIP_4: track 4.07 -> 24.4 mm
- net IR_PWR: track 0.00 -> 19.6 mm
- net DIP_5: track 4.86 -> 18.5 mm
- net N$1: track 0.00 -> 10.1 mm
- net LED_PWR: track 0.00 -> 6.40 mm
- net N$2: track 14.0 -> 11.1 mm
- net DIP_1: track 33.1 -> 30.5 mm
- net N$3: track 2.54 -> 3.81 mm
- net DIP_2: track 24.6 -> 23.8 mm

Commit message: no message
Parts:
- moved LED 1.27 mm to (35.6, 57.8)
- moved R7.680K 1.27 mm to (43.2, 39.4)
- moved R8.680K 1.27 mm to (47.6, 39.4)
- moved R9.680K 1.27 mm to (52.1, 39.4)
- moved U$2 1.27 mm to (51.4, 47.0)
- moved R1.10K 1.27 mm to (62.2, 38.7)
- moved R2.100 1.27 mm to (62.2, 50.8)
- moved R3.39 1.27 mm to (46.4, 58.4)
- moved R4.82 1.27 mm to (34.3, 50.2)
- moved R5.680K 1.27 mm to (34.3, 39.4)
- moved R6.680K 1.27 mm to (38.7, 39.4)
- moved U$1 1.27 mm to (62.2, 56.5)
Connections:
- net DIP_PWR: now also J1.2; no longer J1.3
- net TR_PWR: now also J1.3; no longer J1.2
Routing:
- net DIP_PWR: track 53.9 -> 26.1 mm
- net DIP_5: track 18.5 -> 23.5 mm
- net DIP_4: track 24.4 -> 27.2 mm
- net IR_PWR: track 19.6 -> 17.2 mm
- net DIP_3: track 29.4 -> 31.8 mm
- net TR_PWR: track 34.7 -> 37.0 mm
- net SIG: track 32.9 -> 31.6 mm
- net DIP_2: track 23.8 -> 25.1 mm
- net LED_PWR: track 6.40 -> 7.67 mm
- net DIP_1: track 30.5 -> 31.1 mm
Other:
- board text added: "DIP.1"
- board text added: "DIP.2"
- board text added: "DIP.3"
- board text added: "DIP.4"
- board text added: "DIP.5"
- board text added: "DIP.PWR"
- board text added: "GND"
- board text added: "IR.PWR"
- board text added: "LED.PWR"
- board text added: "SIG"
- board text added: "TR.PWR"
