File: base.brd (EAGLE design)
At the start: 53.3 x 29.2 mm, 16 parts

Commit message: updated layout and part
Parts:
- removed R1.10K: 93PR10KLF, ferraris_sensor_project:93PR10KLF
- added U$3: CT6EP103, ferraris_sensor_project:CT6EP103
- moved LED 33.5 mm to (63.5, 39.4)
- moved R4.82 24.1 mm to (55.9, 39.4)
- moved U$1 9.94 mm to (53.3, 52.1), turned to 90 degrees
- moved U$2 6.35 mm to (45.1, 47.0)
- moved R3.39 4.45 mm to (41.9, 58.4)
- moved R2.100 4.02 mm to (63.5, 47.0)
- moved R5.680K 0.61 mm to (33.7, 39.4)
- moved R6.680K 0.61 mm to (38.1, 39.4)
- moved R7.680K 0.61 mm to (42.6, 39.4)
- moved R8.680K 0.61 mm to (47.0, 39.4)
- moved R9.680K 0.61 mm to (51.5, 39.4)
Connections:
- net N$1: now also U$3.1; no longer R1.10K.1
- net P$1: now also U$3.3; no longer R1.10K.3
- net SIG: now also U$3.2; no longer R1.10K.2
Routing:
- net LED_PWR: track 7.67 -> 31.1 mm
- net DIP_5: track 23.5 -> 12.9 mm
- net DIP_4: track 27.2 -> 16.8 mm
- net DIP_3: track 31.8 -> 23.7 mm
- net TR_PWR: track 37.0 -> 30.4 mm
- net IR_PWR: track 17.2 -> 10.7 mm
- net DIP_PWR: track 26.1 -> 20.5 mm
- net SIG: track 31.6 -> 27.2 mm
- net N$3: track 3.81 -> 7.93 mm
- net DIP_1: track 31.1 -> 33.6 mm
- net DIP_2: track 25.1 -> 26.9 mm
- net N$1: track 10.1 -> 11.3 mm

Commit message: no message
Routing:
- net SIG: track 27.2 -> 26.5 mm
Changed lines of the file:
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@@
 <contactref element="R3.39" pad="1"/>
 <contactref element="J2" pad="2"/>
-<wire x1="27.94" y1="57.15" x2="36.83" y2="57.15" width="0.3048" layer="1"/>
+<wire x1="27.94" y1="57.15" x2="33.655" y2="57.15" width="0.3048" layer="1"/>
+<wire x1="33.655" y1="57.15" x2="36.83" y2="57.15" width="0.3048" layer="1"/>
 <wire x1="36.83" y1="57.15" x2="38.1" y2="58.42" width="0.3048" layer="1"/>
 </signal>
@@
 <contactref element="U$1" pad="3"/>
 <contactref element="J1" pad="3"/>
-<wire x1="54.59" y1="50.82" x2="54.59" y2="48.915" width="0.3048" layer="1"/>
-<wire x1="54.59" y1="48.915" x2="54.61" y2="48.895" width="0.3048" layer="1"/>
-<wire x1="50.8" y1="45.085" x2="54.61" y2="48.895" width="0.3048" layer="1"/>
-<wire x1="30.48" y1="45.72" x2="31.115" y2="45.085" width="0.3048" layer="1"/>
-<wire x1="27.94" y1="45.72" x2="30.48" y2="45.72" width="0.3048" layer="1"/>
-<wire x1="31.115" y1="45.085" x2="50.8" y2="45.085" width="0.3048" layer="1"/>
+<wire x1="54.59" y1="50.82" x2="54.61" y2="50.8" width="0.3048" layer="1"/>
+<wire x1="54.61" y1="50.8" x2="54.61" y2="48.895" width="0.3048" layer="1"/>
+<wire x1="54.61" y1="48.895" x2="50.8" y2="45.085" width="0.3048" layer="1"/>
+<wire x1="31.115" y1="45.085" x2="30.48" y2="45.72" width="0.3048" layer="1"/>
+<wire x1="30.48" y1="45.72" x2="27.94" y2="45.72" width="0.3048" layer="1"/>
+<wire x1="50.8" y1="45.085" x2="31.115" y2="45.085" width="0.3048" layer="1"/>
 </signal>
 <signal name="DIP_3">
@@
 <contactref element="J2" pad="1"/>
 <wire x1="27.94" y1="59.69" x2="29.845" y2="59.69" width="0.3048" layer="16"/>
-<wire x1="29.845" y1="59.69" x2="31.75" y2="57.785" width="0.3048" layer="16"/>
+<wire x1="29.845" y1="59.69" x2="31.115" y2="58.42" width="0.3048" layer="16"/>
+<wire x1="31.115" y1="58.42" x2="31.75" y2="57.785" width="0.3048" layer="16"/>
 <wire x1="31.75" y1="57.785" x2="31.75" y2="55.245" width="0.3048" layer="16"/>
 <wire x1="31.75" y1="55.245" x2="40.005" y2="46.99" width="0.3048" layer="16"/>
@@
 <wire x1="54.59" y1="53.32" x2="54.61" y2="53.34" width="0.3048" layer="16"/>
 <wire x1="54.61" y1="53.34" x2="61" y2="53.34" width="0.3048" layer="16"/>
-<wire x1="61" y1="53.34" x2="61" y2="58.46" width="0.3048" layer="16"/>
-<wire x1="61" y1="58.46" x2="62.23" y2="59.69" width="0.3048" layer="16"/>
-<wire x1="62.23" y1="59.69" x2="76.2" y2="59.69" width="0.3048" layer="16"/>
+<wire x1="61" y1="53.34" x2="61" y2="57.19" width="0.3048" layer="16"/>
+<wire x1="61" y1="57.19" x2="63.5" y2="59.69" width="0.3048" layer="16"/>
+<wire x1="63.5" y1="59.69" x2="76.2" y2="59.69" width="0.3048" layer="16"/>
 </signal>
 <signal name="N$2">

Commit message: fixed
Routing:
- net DIP_1: track 33.6 -> 34.3 mm
- added copper zone on layer 16, net GND_A
- added copper zone on layer 1, net GND_D
- removed copper zone on layer 1, net GND_A
- removed copper zone on layer 16, net GND_D

Commit message: updated for new part
Parts:
- U$1: value DF1BZ-4DP-2.5DSA -> DF1BZ-4DP-2.5DS; device ferraris_sensor_project:DF1BZ-4DP-2.5DSA -> ferraris_sensor_project:DF1BZ-4DP-2.5DS
- moved U$1 0.36 mm to (53.6, 52.3), turned to 180 degrees
- turned U$3 to 0 degrees
Connections:
- net N$2: now also U$1.4; no longer U$1.1
- net SIG: now also U$1.3; no longer U$1.4
- net TR_PWR: now also U$1.1; no longer U$1.3
Routing:
- net N$1: track 11.3 -> 6.96 mm
- net N$2: track 11.4 -> 8.63 mm
- net SIG: track 26.5 -> 23.9 mm
- net TR_PWR: track 30.4 -> 32.3 mm
Changed lines of the file:
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@@
 <?xml version="1.0" encoding="utf-8"?>
 <!DOCTYPE eagle SYSTEM "eagle.dtd">
-<eagle version="8.7.1">
+<eagle version="9.0.1">
 <drawing>
 <settings>
@@
 <layers>
 <layer number="1" name="Top" color="4" fill="1" visible="yes" active="yes"/>
+<layer number="2" name="Route2" color="1" fill="3" visible="no" active="no"/>
+<layer number="3" name="Route3" color="4" fill="3" visible="no" active="no"/>
+<layer number="4" name="Route4" color="1" fill="4" visible="no" active="no"/>
+<layer number="5" name="Route5" color="4" fill="4" visible="no" active="no"/>
+<layer number="6" name="Route6" color="1" fill="8" visible="no" active="no"/>
+<layer number="7" name="Route7" color="4" fill="8" visible="no" active="no"/>
+<layer number="8" name="Route8" color="1" fill="2" visible="no" active="no"/>
+<layer number="9" name="Route9" color="4" fill="2" visible="no" active="no"/>
+<layer number="10" name="Route10" color="1" fill="7" visible="no" active="no"/>
+<layer number="11" name="Route11" color="4" fill="7" visible="no" active="no"/>
+<layer number="12" name="Route12" color="1" fill="5" visible="no" active="no"/>
+<layer number="13" name="Route13" color="4" fill="5" visible="no" active="no"/>
+<layer number="14" name="Route14" color="1" fill="6" visible="no" active="no"/>
+<layer number="15" name="Route15" color="4" fill="6" visible="no" active="no"/>
 <layer number="16" name="Bottom" color="1" fill="1" visible="yes" active="yes"/>
 <layer number="17" name="Pads" color="2" fill="1" visible="yes" active="yes"/>
@@
 </class>
 </classes>
-<designrules name="aisler_go_2layer">
+<designrules name="aisler_go_2layer *">
 <description language="de">&lt;b&gt;EAGLE Design Rules&lt;/b&gt;
 &lt;p&gt;
@@
 <param name="rlMinPadInner" value="0.25mm"/>
 <param name="rlMaxPadInner" value="100mm"/>
-<param name="rlMinPadBottom" value="0.25mm"/>
+<param name="rlMinPadBottom" value="0.4mm"/>
 <param name="rlMaxPadBottom" value="100mm"/>
 <param name="rlMinViaOuter" value="0.05mm"/>
@@
 <attribute name="SPICEPREFIX" value="R" x="51.4604" y="39.37" size="1.778" layer="27" rot="R270" display="off"/>
 </element>
-<element name="U$1" library="ferraris_sensor_project" package="DF1BZ-4DP-2.5DSA" value="DF1BZ-4DP-2.5DSA" x="53.34" y="52.07" rot="R90"/>
+<element name="U$1" library="ferraris_sensor_project" package="DF1BZ-4DP-2.5DS" value="DF1BZ-4DP-2.5DS" x="53.594" y="52.324" rot="R180"/>
 <element name="U$2" library="ferraris_sensor_project" package="DIP-SW-CTS-208-5" value="DIP-SW-CTS-208-5" x="45.085" y="46.99" rot="R180"/>
-<element name="U$3" library="ferraris_sensor_project" package="CT6EP103" value="CT6EP103" x="63.5" y="53.34" rot="R90"/>
+<element name="U$3" library="ferraris_sensor_project" package="CT6EP103" value="CT6EP103" x="63.5" y="53.34"/>
 </elements>
 <signals>
@@
 <contactref element="J1" pad="3"/>
 <wire x1="31.115" y1="45.085" x2="30.48" y2="45.72" width="0.3048" layer="1"/>
-<wire x1="30.48" y1="45.72" x2="29.845" y2="45.72" width="0.3048" layer="1"/>
-<wire x1="29.845" y1="45.72" x2="27.94" y2="45.72" width="0.3048" layer="1"/>
-<wire x1="31.115" y1="45.085" x2="50.8" y2="45.085" width="0.3048" layer="1"/>
-<contactref element="U$1" pad="3"/>
-<wire x1="50.8" y1="45.085" x2="54.59" y2="48.875" width="0.3048" layer="1"/>
-<wire x1="54.59" y1="48.875" x2="54.59" y2="50.82" width="0.3048" layer="1"/>
+<wire x1="30.48" y1="45.72" x2="27.94" y2="45.72" width="0.3048" layer="1"/>
+<contactref element="U$1" pad="1"/>
+<wire x1="54.844" y1="51.074" x2="54.844" y2="46.589" width="0.3048" layer="1"/>
+<wire x1="54.844" y1="46.589" x2="53.34" y2="45.085" width="0.3048" layer="1"/>
+<wire x1="53.34" y1="45.085" x2="31.115" y2="45.085" width="0.3048" layer="1"/>
 </signal>
 <signal name="DIP_3">
@@
 <contactref element="J3" pad="1"/>
 <contactref element="R2.100" pad="2"/>
-<polygon width="0.1524" layer="16" isolate="0.4064">
+<polygon width="0.1524" layer="16" isolate="0.4064" orphans="yes">
 <vertex x="26.67" y="62.23"/>
 <vertex x="77.47" y="62.23"/>
@@
 <contactref element="J4" pad="1"/>
 <contactref element="U$3" pad="2"/>
-<contactref element="U$1" pad="4"/>
-<wire x1="54.59" y1="53.32" x2="54.61" y2="53.34" width="0.3048" layer="1"/>
-<wire x1="54.61" y1="53.34" x2="61" y2="53.34" width="0.3048" layer="1"/>
-<wire x1="61" y1="53.34" x2="60.96" y2="53.38" width="0.3048" layer="1"/>
-<wire x1="60.96" y1="53.38" x2="60.96" y2="57.15" width="0.3048" layer="1"/>
-<wire x1="60.96" y1="57.15" x2="63.5" y2="59.69" width="0.3048" layer="1"/>
-<wire x1="63.5" y1="59.69" x2="76.2" y2="59.69" width="0.3048" layer="1"/>
-</signal>
-<signal name="N$2">
-<contactref element="R3.39" pad="2"/>
-<contactref element="U$1" pad="1"/>
-<wire x1="45.72" y1="58.42" x2="48.895" y2="55.245" width="0.3048" layer="1"/>
-<wire x1="48.895" y1="55.245" x2="48.895" y2="52.07" width="0.3048" layer="1"/>
-<wire x1="48.895" y1="52.07" x2="50.165" y2="50.8" width="0.3048" layer="1"/>
-<wire x1="50.165" y1="50.8" x2="52.07" y2="50.8" width="0.3048" layer="1"/>
-<wire x1="52.07" y1="50.8" x2="52.09" y2="50.82" width="0.3048" layer="1"/>
+<wire x1="63.5" y1="55.84" x2="67.35" y2="59.69" width="0.3048" layer="1"/>
+<wire x1="67.35" y1="59.69" x2="76.2" y2="59.69" width="0.3048" layer="1"/>
+<contactref element="U$1" pad="3"/>
+<wire x1="63.5" y1="55.84" x2="57.11" y2="55.84" width="0.3048" layer="1"/>
+<wire x1="57.11" y1="55.84" x2="54.844" y2="53.574" width="0.3048" layer="1"/>
 </signal>
 <signal name="N$1">
 <contactref element="R2.100" pad="1"/>
 <contactref element="U$3" pad="1"/>
-<wire x1="63.46" y1="55.78" x2="63.56" y2="55.88" width="0.3048" layer="1"/>
-<wire x1="63.56" y1="55.88" x2="64.77" y2="55.88" width="0.3048" layer="1"/>
-<wire x1="64.77" y1="55.88" x2="67.31" y2="53.34" width="0.3048" layer="1"/>
-<wire x1="67.31" y1="53.34" x2="67.31" y2="46.99" width="0.3048" layer="1"/>
+<wire x1="65.94" y1="53.38" x2="67.31" y2="52.01" width="0.3048" layer="1"/>
+<wire x1="67.31" y1="52.01" x2="67.31" y2="46.99" width="0.3048" layer="1"/>
+</signal>
+<signal name="N$2">
+<contactref element="R3.39" pad="2"/>
+<contactref element="U$1" pad="4"/>
+<wire x1="52.344" y1="53.574" x2="50.566" y2="53.574" width="0.3048" layer="1"/>
+<wire x1="50.566" y1="53.574" x2="45.72" y2="58.42" width="0.3048" layer="1"/>
 </signal>
 </signals>

Commit message: fixes
Connections:
- net GND_D: now also U$1.1; no longer U$1.2
- net TR_PWR: now also U$1.2; no longer U$1.1
Routing:
- net TR_PWR: track 32.3 -> 27.1 mm
Changed lines of the file:
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@@
 <contactref element="R4.82" pad="2"/>
 <contactref element="LED" pad="A"/>
-<wire x1="55.88" y1="43.18" x2="57.15" y2="43.18" width="0.3048" layer="1"/>
-<wire x1="57.15" y1="43.18" x2="60.96" y2="39.37" width="0.3048" layer="1"/>
-<wire x1="60.96" y1="39.37" x2="62.23" y2="39.37" width="0.3048" layer="1"/>
+<wire x1="55.88" y1="43.18" x2="59.69" y2="39.37" width="0.3048" layer="1"/>
+<wire x1="59.69" y1="39.37" x2="62.23" y2="39.37" width="0.3048" layer="1"/>
 </signal>
 <signal name="GND_D">
@@
 <contactref element="R9.680K" pad="2"/>
 <contactref element="LED" pad="K"/>
-<contactref element="U$1" pad="2"/>
 <polygon width="0.1524" layer="1" isolate="0.4064">
 <vertex x="26.67" y="62.23"/>
@@
 <vertex x="25.4" y="60.96"/>
 </polygon>
+<contactref element="U$1" pad="1"/>
 </signal>
 <signal name="DIP_1">
@@
 <signal name="TR_PWR">
 <contactref element="J1" pad="3"/>
-<wire x1="31.115" y1="45.085" x2="30.48" y2="45.72" width="0.3048" layer="1"/>
-<wire x1="30.48" y1="45.72" x2="27.94" y2="45.72" width="0.3048" layer="1"/>
-<contactref element="U$1" pad="1"/>
-<wire x1="54.844" y1="51.074" x2="54.844" y2="46.589" width="0.3048" layer="1"/>
-<wire x1="54.844" y1="46.589" x2="53.34" y2="45.085" width="0.3048" layer="1"/>
-<wire x1="53.34" y1="45.085" x2="31.115" y2="45.085" width="0.3048" layer="1"/>
+<contactref element="U$1" pad="2"/>
+<wire x1="46.355" y1="45.085" x2="52.344" y2="51.074" width="0.3048" layer="1"/>
+<wire x1="27.94" y1="45.72" x2="29.845" y2="45.72" width="0.3048" layer="1"/>
+<wire x1="29.845" y1="45.72" x2="30.48" y2="45.085" width="0.3048" layer="1"/>
+<wire x1="30.48" y1="45.085" x2="46.355" y2="45.085" width="0.3048" layer="1"/>
 </signal>
 <signal name="DIP_3">
