File: head.brd (EAGLE design)
At the start: 63.5 x 12.7 mm, 6 parts

Commit message: fixed
Parts:
- moved 2 6.60 mm to (50.4, 33.1)
- moved 4 6.60 mm to (57.0, 33.1)
Connections:
- net GND_A: now also 4.1; no longer 3.1
- net TR_PWR: now also 3.1; no longer 4.1
Routing:
- net TR_PWR: track 5.03 -> 6.46 mm
Other:
- board text added: "GND"
- board text added: "IR_PWR"
- board text added: "SIG/GND"
- board text added: "TR_PWR"
Changed lines of the file:
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@@
 <drawing>
 <settings>
-<setting alwaysvectorfont="yes"/>
+<setting alwaysvectorfont="no"/>
 <setting verticaltext="up"/>
 </settings>
@@
 <wire x1="20.955" y1="39.37" x2="83.185" y2="39.37" width="0.1524" layer="26"/>
 <text x="25.2222" y="40.9956" size="1.27" layer="26" rot="MR0">SEPL</text>
+<text x="46.101" y="31.242" size="0.4064" layer="25">IR_PWR</text>
+<text x="52.6034" y="31.242" size="0.4064" layer="25">TR_PWR</text>
+<text x="49.7332" y="31.242" size="0.4064" layer="25">GND</text>
+<text x="55.7784" y="31.242" size="0.4064" layer="25">SIG/GND</text>
 </plain>
 <attributes>
@@
 <elements>
 <element name="1" library="wirepad" library_urn="urn:adsk.eagle:library:412" package="2,15/1,0" package3d_urn="urn:adsk.eagle:package:30831/1" value="" x="47.1805" y="33.147"/>
-<element name="2" library="wirepad" library_urn="urn:adsk.eagle:library:412" package="2,15/1,0" package3d_urn="urn:adsk.eagle:package:30831/1" value="" x="56.9595" y="33.147"/>
+<element name="2" library="wirepad" library_urn="urn:adsk.eagle:library:412" package="2,15/1,0" package3d_urn="urn:adsk.eagle:package:30831/1" value="" x="50.3555" y="33.147"/>
+<element name="4" library="wirepad" library_urn="urn:adsk.eagle:library:412" package="2,15/1,0" package3d_urn="urn:adsk.eagle:package:30831/1" value="" x="56.9595" y="33.147"/>
 <element name="3" library="wirepad" library_urn="urn:adsk.eagle:library:412" package="2,15/1,0" package3d_urn="urn:adsk.eagle:package:30831/1" value="" x="53.7972" y="33.147"/>
-<element name="4" library="wirepad" library_urn="urn:adsk.eagle:library:412" package="2,15/1,0" package3d_urn="urn:adsk.eagle:package:30831/1" value="" x="50.3555" y="33.147"/>
 <element name="U$1" library="ferraris_sensor_project" package="CNY70" value="CNY70" x="48.4505" y="39.37"/>
 <element name="U$2" library="ferraris_sensor_project" package="CNY70" value="CNY70" x="55.6895" y="39.37" rot="R180"/>
@@
 <signal name="TR_PWR">
 <contactref element="U$1" pad="COLL"/>
-<contactref element="4" pad="1"/>
-<wire x1="49.8505" y1="37.97" x2="49.8505" y2="35.9507" width="0.3048" layer="1"/>
-<wire x1="49.8505" y1="35.9507" x2="50.3428" y2="35.4584" width="0.3048" layer="1"/>
-<wire x1="50.3428" y1="35.4584" x2="50.3428" y2="33.1597" width="0.3048" layer="1"/>
-<wire x1="50.3428" y1="33.1597" x2="50.3555" y2="33.147" width="0.3048" layer="1"/>
+<contactref element="3" pad="1"/>
+<wire x1="49.8505" y1="37.97" x2="49.8505" y2="37.0937" width="0.3048" layer="1"/>
+<wire x1="49.8505" y1="37.0937" x2="53.7972" y2="33.147" width="0.3048" layer="1"/>
 </signal>
 <signal name="GND_A">
 <contactref element="U$2" pad="E"/>
-<contactref element="3" pad="1"/>
+<contactref element="4" pad="1"/>
 <polygon width="0.1524" layer="16" isolate="0.4064">
 <vertex x="44.45" y="41.91"/>

Commit message: updated for new part
Parts:
- moved 4 9.78 mm to (47.2, 33.1)
- moved 1 6.62 mm to (53.8, 33.1)
- moved 2 6.60 mm to (57.0, 33.1)
- moved 3 3.44 mm to (50.4, 33.1)
Connections:
- net GND_A: now also 3.1; no longer 4.1
- net IR_PWR: now also 4.1; no longer 1.1
- net TR_PWR: now also 1.1; no longer 3.1
Other:
- board size 63.5 x 12.7 mm -> 63.5 x 17.8 mm
- board text added: "SIG"
- board text removed: "SIG/GND"
Changed lines of the file:
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@@
 <?xml version="1.0" encoding="utf-8"?>
 <!DOCTYPE eagle SYSTEM "eagle.dtd">
-<eagle version="8.7.1">
+<eagle version="9.0.1">
 <drawing>
 <settings>
-<setting alwaysvectorfont="no"/>
+<setting alwaysvectorfont="yes"/>
 <setting verticaltext="up"/>
 </settings>
@@
 <layers>
 <layer number="1" name="Top" color="4" fill="1" visible="yes" active="yes"/>
+<layer number="2" name="Route2" color="1" fill="3" visible="no" active="no"/>
+<layer number="3" name="Route3" color="4" fill="3" visible="no" active="no"/>
+<layer number="4" name="Route4" color="1" fill="4" visible="no" active="no"/>
+<layer number="5" name="Route5" color="4" fill="4" visible="no" active="no"/>
+<layer number="6" name="Route6" color="1" fill="8" visible="no" active="no"/>
+<layer number="7" name="Route7" color="4" fill="8" visible="no" active="no"/>
+<layer number="8" name="Route8" color="1" fill="2" visible="no" active="no"/>
+<layer number="9" name="Route9" color="4" fill="2" visible="no" active="no"/>
+<layer number="10" name="Route10" color="1" fill="7" visible="no" active="no"/>
+<layer number="11" name="Route11" color="4" fill="7" visible="no" active="no"/>
+<layer number="12" name="Route12" color="1" fill="5" visible="no" active="no"/>
+<layer number="13" name="Route13" color="4" fill="5" visible="no" active="no"/>
+<layer number="14" name="Route14" color="1" fill="6" visible="no" active="no"/>
+<layer number="15" name="Route15" color="4" fill="6" visible="no" active="no"/>
 <layer number="16" name="Bottom" color="1" fill="1" visible="yes" active="yes"/>
 <layer number="17" name="Pads" color="2" fill="1" visible="yes" active="yes"/>
@@
 <wire x1="20.32" y1="36.83" x2="20.32" y2="41.91" width="0.1524" layer="20"/>
 <wire x1="21.59" y1="35.56" x2="43.18" y2="35.56" width="0.1524" layer="20"/>
-<wire x1="43.18" y1="35.56" x2="44.45" y2="34.29" width="0.1524" layer="20"/>
-<wire x1="44.45" y1="34.29" x2="44.45" y2="31.75" width="0.1524" layer="20"/>
-<wire x1="44.45" y1="31.75" x2="45.72" y2="30.48" width="0.1524" layer="20"/>
-<wire x1="45.72" y1="30.48" x2="58.42" y2="30.48" width="0.1524" layer="20"/>
+<hole x="39.3954" y="39.37" drill="2.032"/>
+<hole x="64.77" y="39.37" drill="2.032"/>
+<wire x1="60.96" y1="35.56" x2="82.55" y2="35.56" width="0.1524" layer="20"/>
+<wire x1="20.955" y1="39.37" x2="83.185" y2="39.37" width="0.1524" layer="26"/>
+<text x="25.2222" y="40.9956" size="1.27" layer="26" rot="MR0">SEPL</text>
+<text x="45.72" y="30.988" size="0.6096" layer="25">IR_PWR</text>
+<text x="52.2224" y="30.988" size="0.6096" layer="25">TR_PWR</text>
+<text x="56.2102" y="30.988" size="0.6096" layer="25">GND</text>
+<text x="49.6824" y="30.988" size="0.6096" layer="25">SIG</text>
+<wire x1="48.26" y1="26.67" x2="49.53" y2="25.4" width="0.1524" layer="20"/>
+<wire x1="49.53" y1="25.4" x2="54.61" y2="25.4" width="0.1524" layer="20"/>
+<wire x1="54.61" y1="25.4" x2="55.88" y2="26.67" width="0.1524" layer="20"/>
+<wire x1="46.99" y1="30.48" x2="48.26" y2="29.21" width="0.1524" layer="20"/>
+<wire x1="48.26" y1="29.21" x2="48.26" y2="26.67" width="0.1524" layer="20"/>
+<wire x1="46.99" y1="30.48" x2="45.72" y2="30.48" width="0.1524" layer="20"/>
+<wire x1="55.88" y1="29.21" x2="57.15" y2="30.48" width="0.1524" layer="20"/>
+<wire x1="57.15" y1="30.48" x2="58.42" y2="30.48" width="0.1524" layer="20"/>
+<wire x1="55.88" y1="29.21" x2="55.88" y2="26.67" width="0.1524" layer="20"/>
+<wire x1="52.07" y1="26.035" x2="52.07" y2="42.545" width="0.1524" layer="26"/>
+<wire x1="45.72" y1="30.48" x2="44.45" y2="31.75" width="0.1524" layer="20"/>
+<wire x1="44.45" y1="31.75" x2="44.45" y2="34.29" width="0.1524" layer="20"/>
+<wire x1="44.45" y1="34.29" x2="43.18" y2="35.56" width="0.1524" layer="20"/>
 <wire x1="58.42" y1="30.48" x2="59.69" y2="31.75" width="0.1524" layer="20"/>
 <wire x1="59.69" y1="31.75" x2="59.69" y2="34.29" width="0.1524" layer="20"/>
 <wire x1="59.69" y1="34.29" x2="60.96" y2="35.56" width="0.1524" layer="20"/>
-<wire x1="60.96" y1="35.56" x2="82.55" y2="35.56" width="0.1524" layer="20"/>
-<wire x1="52.07" y1="42.545" x2="52.07" y2="31.115" width="0.1524" layer="26"/>
-<hole x="39.3954" y="39.37" drill="2.032"/>
-<hole x="64.77" y="39.37" drill="2.032"/>
-<wire x1="20.955" y1="39.37" x2="83.185" y2="39.37" width="0.1524" layer="26"/>
-<text x="25.2222" y="40.9956" size="1.27" layer="26" rot="MR0">SEPL</text>
-<text x="46.101" y="31.242" size="0.4064" layer="25">IR_PWR</text>
-<text x="52.6034" y="31.242" size="0.4064" layer="25">TR_PWR</text>
-<text x="49.7332" y="31.242" size="0.4064" layer="25">GND</text>
-<text x="55.7784" y="31.242" size="0.4064" layer="25">SIG/GND</text>
 </plain>
 <attributes>
@@
 </class>
 </classes>
-<designrules name="aisler_go_2layer">
+<designrules name="aisler_go_2layer *">
 <description language="de">&lt;b&gt;EAGLE Design Rules&lt;/b&gt;
 &lt;p&gt;
@@
 <param name="rlMinPadInner" value="0.25mm"/>
 <param name="rlMaxPadInner" value="100mm"/>
-<param name="rlMinPadBottom" value="0.25mm"/>
+<param name="rlMinPadBottom" value="0.4mm"/>
 <param name="rlMaxPadBottom" value="100mm"/>
 <param name="rlMinViaOuter" value="0.05mm"/>
@@
 </autorouter>
 <elements>
-<element name="1" library="wirepad" library_urn="urn:adsk.eagle:library:412" package="2,15/1,0" package3d_urn="urn:adsk.eagle:package:30831/1" value="" x="47.1805" y="33.147"/>
-<element name="2" library="wirepad" library_urn="urn:adsk.eagle:library:412" package="2,15/1,0" package3d_urn="urn:adsk.eagle:package:30831/1" value="" x="50.3555" y="33.147"/>
-<element name="4" library="wirepad" library_urn="urn:adsk.eagle:library:412" package="2,15/1,0" package3d_urn="urn:adsk.eagle:package:30831/1" value="" x="56.9595" y="33.147"/>
-<element name="3" library="wirepad" library_urn="urn:adsk.eagle:library:412" package="2,15/1,0" package3d_urn="urn:adsk.eagle:package:30831/1" value="" x="53.7972" y="33.147"/>
+<element name="4" library="wirepad" library_urn="urn:adsk.eagle:library:412" package="2,15/1,0" package3d_urn="urn:adsk.eagle:package:30831/1" value="" x="47.1805" y="33.147"/>
+<element name="2" library="wirepad" library_urn="urn:adsk.eagle:library:412" package="2,15/1,0" package3d_urn="urn:adsk.eagle:package:30831/1" value="" x="56.9595" y="33.147"/>
+<element name="3" library="wirepad" library_urn="urn:adsk.eagle:library:412" package="2,15/1,0" package3d_urn="urn:adsk.eagle:package:30831/1" value="" x="50.3555" y="33.147"/>
+<element name="1" library="wirepad" library_urn="urn:adsk.eagle:library:412" package="2,15/1,0" package3d_urn="urn:adsk.eagle:package:30831/1" value="" x="53.7972" y="33.147"/>
 <element name="U$1" library="ferraris_sensor_project" package="CNY70" value="CNY70" x="48.4505" y="39.37"/>
 <element name="U$2" library="ferraris_sensor_project" package="CNY70" value="CNY70" x="55.6895" y="39.37" rot="R180"/>
@@
 <signal name="TR_PWR">
 <contactref element="U$1" pad="COLL"/>
-<contactref element="3" pad="1"/>
+<contactref element="1" pad="1"/>
 <wire x1="49.8505" y1="37.97" x2="49.8505" y2="37.0937" width="0.3048" layer="1"/>
 <wire x1="49.8505" y1="37.0937" x2="53.7972" y2="33.147" width="0.3048" layer="1"/>
@@
 <signal name="GND_A">
 <contactref element="U$2" pad="E"/>
-<contactref element="4" pad="1"/>
+<contactref element="3" pad="1"/>
 <polygon width="0.1524" layer="16" isolate="0.4064">
 <vertex x="44.45" y="41.91"/>
@@
 </signal>
 <signal name="IR_PWR">
-<contactref element="1" pad="1"/>
+<contactref element="4" pad="1"/>
 <contactref element="U$2" pad="A"/>
 <contactref element="U$1" pad="A"/>

Commit message: fixes
Parts:
- moved 1 3.16 mm to (57.0, 33.1)
- moved 2 3.16 mm to (53.8, 33.1)
Connections:
- net GND_D: now also 1.1; no longer 2.1
- net TR_PWR: now also 2.1; no longer 1.1
Other:
- outline, holes or cut-outs redrawn
Changed lines of the file:
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@@
 <wire x1="21.59" y1="35.56" x2="20.32" y2="36.83" width="0.1524" layer="20"/>
 <wire x1="20.32" y1="36.83" x2="20.32" y2="41.91" width="0.1524" layer="20"/>
-<wire x1="21.59" y1="35.56" x2="43.18" y2="35.56" width="0.1524" layer="20"/>
+<wire x1="21.59" y1="35.56" x2="42.545" y2="35.56" width="0.1524" layer="20"/>
 <hole x="39.3954" y="39.37" drill="2.032"/>
 <hole x="64.77" y="39.37" drill="2.032"/>
-<wire x1="60.96" y1="35.56" x2="82.55" y2="35.56" width="0.1524" layer="20"/>
+<wire x1="61.595" y1="35.56" x2="82.55" y2="35.56" width="0.1524" layer="20"/>
 <wire x1="20.955" y1="39.37" x2="83.185" y2="39.37" width="0.1524" layer="26"/>
-<text x="25.2222" y="40.9956" size="1.27" layer="26" rot="MR0">SEPL</text>
+<text x="53.975" y="27.0256" size="1.27" layer="26" rot="MR0">SEPL</text>
 <text x="45.72" y="30.988" size="0.6096" layer="25">IR_PWR</text>
 <text x="52.2224" y="30.988" size="0.6096" layer="25">TR_PWR</text>
@@
 <wire x1="49.53" y1="25.4" x2="54.61" y2="25.4" width="0.1524" layer="20"/>
 <wire x1="54.61" y1="25.4" x2="55.88" y2="26.67" width="0.1524" layer="20"/>
-<wire x1="46.99" y1="30.48" x2="48.26" y2="29.21" width="0.1524" layer="20"/>
-<wire x1="48.26" y1="29.21" x2="48.26" y2="26.67" width="0.1524" layer="20"/>
-<wire x1="46.99" y1="30.48" x2="45.72" y2="30.48" width="0.1524" layer="20"/>
-<wire x1="55.88" y1="29.21" x2="57.15" y2="30.48" width="0.1524" layer="20"/>
-<wire x1="57.15" y1="30.48" x2="58.42" y2="30.48" width="0.1524" layer="20"/>
-<wire x1="55.88" y1="29.21" x2="55.88" y2="26.67" width="0.1524" layer="20"/>
-<wire x1="52.07" y1="26.035" x2="52.07" y2="42.545" width="0.1524" layer="26"/>
-<wire x1="45.72" y1="30.48" x2="44.45" y2="31.75" width="0.1524" layer="20"/>
-<wire x1="44.45" y1="31.75" x2="44.45" y2="34.29" width="0.1524" layer="20"/>
-<wire x1="44.45" y1="34.29" x2="43.18" y2="35.56" width="0.1524" layer="20"/>
-<wire x1="58.42" y1="30.48" x2="59.69" y2="31.75" width="0.1524" layer="20"/>
-<wire x1="59.69" y1="31.75" x2="59.69" y2="34.29" width="0.1524" layer="20"/>
-<wire x1="59.69" y1="34.29" x2="60.96" y2="35.56" width="0.1524" layer="20"/>
+<wire x1="52.07" y1="42.545" x2="52.07" y2="29.21" width="0.1524" layer="26"/>
+<wire x1="60.325" y1="34.29" x2="61.595" y2="35.56" width="0.1524" layer="20"/>
+<wire x1="60.325" y1="34.29" x2="60.325" y2="31.115" width="0.1524" layer="20"/>
+<wire x1="60.325" y1="31.115" x2="59.055" y2="29.845" width="0.1524" layer="20"/>
+<wire x1="42.545" y1="35.56" x2="43.815" y2="34.29" width="0.1524" layer="20"/>
+<wire x1="43.815" y1="34.29" x2="43.815" y2="31.115" width="0.1524" layer="20"/>
+<wire x1="43.815" y1="31.115" x2="45.085" y2="29.845" width="0.1524" layer="20"/>
+<wire x1="45.085" y1="29.845" x2="46.99" y2="29.845" width="0.1524" layer="20"/>
+<wire x1="46.99" y1="29.845" x2="48.26" y2="28.575" width="0.1524" layer="20"/>
+<wire x1="48.26" y1="28.575" x2="48.26" y2="26.67" width="0.1524" layer="20"/>
+<wire x1="55.88" y1="26.67" x2="55.88" y2="28.575" width="0.1524" layer="20"/>
+<wire x1="55.88" y1="28.575" x2="57.15" y2="29.845" width="0.1524" layer="20"/>
+<wire x1="57.15" y1="29.845" x2="59.055" y2="29.845" width="0.1524" layer="20"/>
 </plain>
 <attributes>
@@
 <elements>
 <element name="4" library="wirepad" library_urn="urn:adsk.eagle:library:412" package="2,15/1,0" package3d_urn="urn:adsk.eagle:package:30831/1" value="" x="47.1805" y="33.147"/>
-<element name="2" library="wirepad" library_urn="urn:adsk.eagle:library:412" package="2,15/1,0" package3d_urn="urn:adsk.eagle:package:30831/1" value="" x="56.9595" y="33.147"/>
+<element name="1" library="wirepad" library_urn="urn:adsk.eagle:library:412" package="2,15/1,0" package3d_urn="urn:adsk.eagle:package:30831/1" value="" x="56.9595" y="33.147"/>
 <element name="3" library="wirepad" library_urn="urn:adsk.eagle:library:412" package="2,15/1,0" package3d_urn="urn:adsk.eagle:package:30831/1" value="" x="50.3555" y="33.147"/>
-<element name="1" library="wirepad" library_urn="urn:adsk.eagle:library:412" package="2,15/1,0" package3d_urn="urn:adsk.eagle:package:30831/1" value="" x="53.7972" y="33.147"/>
+<element name="2" library="wirepad" library_urn="urn:adsk.eagle:library:412" package="2,15/1,0" package3d_urn="urn:adsk.eagle:package:30831/1" value="" x="53.7972" y="33.147"/>
 <element name="U$1" library="ferraris_sensor_project" package="CNY70" value="CNY70" x="48.4505" y="39.37"/>
 <element name="U$2" library="ferraris_sensor_project" package="CNY70" value="CNY70" x="55.6895" y="39.37" rot="R180"/>
@@
 <signal name="GND_D">
 <contactref element="U$2" pad="CATH"/>
-<contactref element="2" pad="1"/>
+<contactref element="1" pad="1"/>
 <contactref element="U$1" pad="CATH"/>
 <polygon width="0.1524" layer="1" isolate="0.4064">
@@
 <signal name="TR_PWR">
 <contactref element="U$1" pad="COLL"/>
-<contactref element="1" pad="1"/>
+<contactref element="2" pad="1"/>
 <wire x1="49.8505" y1="37.97" x2="49.8505" y2="37.0937" width="0.3048" layer="1"/>
 <wire x1="49.8505" y1="37.0937" x2="53.7972" y2="33.147" width="0.3048" layer="1"/>
