File: head.sch (EAGLE design)
At the start: 6 parts

Commit message: no message
Parts:
- renumbered A(5V) to 1, CATH(GND) to 2, COLL(5V) to 4, E(SIG+GND) to 3
Changed lines of the file:
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@@
 <part name="U$1" library="ferraris_sensor_project" deviceset="CNY70" device=""/>
 <part name="U$2" library="ferraris_sensor_project" deviceset="CNY70" device=""/>
-<part name="A(5V)" library="wirepad" library_urn="urn:adsk.eagle:library:412" deviceset="2,15/1,0" device="" package3d_urn="urn:adsk.eagle:package:30831/1"/>
-<part name="CATH(GND)" library="wirepad" library_urn="urn:adsk.eagle:library:412" deviceset="2,15/1,0" device="" package3d_urn="urn:adsk.eagle:package:30831/1"/>
-<part name="COLL(5V)" library="wirepad" library_urn="urn:adsk.eagle:library:412" deviceset="2,15/1,0" device="" package3d_urn="urn:adsk.eagle:package:30831/1"/>
-<part name="E(SIG+GND)" library="wirepad" library_urn="urn:adsk.eagle:library:412" deviceset="2,15/1,0" device="" package3d_urn="urn:adsk.eagle:package:30831/1"/>
+<part name="1" library="wirepad" library_urn="urn:adsk.eagle:library:412" deviceset="2,15/1,0" device="" package3d_urn="urn:adsk.eagle:package:30831/1"/>
+<part name="2" library="wirepad" library_urn="urn:adsk.eagle:library:412" deviceset="2,15/1,0" device="" package3d_urn="urn:adsk.eagle:package:30831/1"/>
+<part name="4" library="wirepad" library_urn="urn:adsk.eagle:library:412" deviceset="2,15/1,0" device="" package3d_urn="urn:adsk.eagle:package:30831/1"/>
+<part name="3" library="wirepad" library_urn="urn:adsk.eagle:library:412" deviceset="2,15/1,0" device="" package3d_urn="urn:adsk.eagle:package:30831/1"/>
 </parts>
 <sheets>
@@
 <instance part="U$1" gate="G$1" x="60.96" y="58.42"/>
 <instance part="U$2" gate="G$1" x="81.28" y="58.42" rot="R180"/>
-<instance part="A(5V)" gate="1" x="68.58" y="71.12"/>
-<instance part="CATH(GND)" gate="1" x="73.66" y="30.48" rot="R180"/>
-<instance part="COLL(5V)" gate="1" x="55.88" y="48.26"/>
-<instance part="E(SIG+GND)" gate="1" x="55.88" y="40.64"/>
+<instance part="1" gate="1" x="68.58" y="71.12"/>
+<instance part="2" gate="1" x="73.66" y="30.48" rot="R180"/>
+<instance part="4" gate="1" x="55.88" y="48.26"/>
+<instance part="3" gate="1" x="55.88" y="40.64"/>
 </instances>
 <busses>
@@
 <wire x1="91.44" y1="35.56" x2="71.12" y2="35.56" width="0.1524" layer="91"/>
 <wire x1="71.12" y1="35.56" x2="50.8" y2="35.56" width="0.1524" layer="91"/>
-<pinref part="CATH(GND)" gate="1" pin="P"/>
+<pinref part="2" gate="1" pin="P"/>
 <wire x1="71.12" y1="30.48" x2="71.12" y2="35.56" width="0.1524" layer="91"/>
 <junction x="71.12" y="35.56"/>
@@
 <segment>
 <pinref part="U$1" gate="G$1" pin="5V(PWR)"/>
-<pinref part="COLL(5V)" gate="1" pin="P"/>
+<pinref part="4" gate="1" pin="P"/>
 <wire x1="67.46" y1="56.92" x2="67.46" y2="48.26" width="0.1524" layer="91"/>
 <wire x1="67.46" y1="48.26" x2="58.42" y2="48.26" width="0.1524" layer="91"/>
@@
 <segment>
 <pinref part="U$2" gate="G$1" pin="GND(PWR)"/>
-<pinref part="E(SIG+GND)" gate="1" pin="P"/>
+<pinref part="3" gate="1" pin="P"/>
 <wire x1="74.78" y1="56.92" x2="74.78" y2="40.64" width="0.1524" layer="91"/>
 <wire x1="74.78" y1="40.64" x2="58.42" y2="40.64" width="0.1524" layer="91"/>
@@
 <net name="A(5V)" class="0">
 <segment>
-<pinref part="A(5V)" gate="1" pin="P"/>
+<pinref part="1" gate="1" pin="P"/>
 <wire x1="71.12" y1="71.12" x2="71.12" y2="66.04" width="0.1524" layer="91"/>
 <wire x1="71.12" y1="66.04" x2="93.98" y2="66.04" width="0.1524" layer="91"/>

Commit message: no message
Connections:
- net A(5V) renamed IR_PWR
- net CATH(GND) renamed GND_D
- net COLL(5V) renamed TR_PWR
- net E(SIG+GND) renamed GND_A
Changed lines of the file:
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@@
 </segment>
 </net>
-<net name="CATH(GND)" class="0">
+<net name="GND_D" class="0">
 <segment>
 <pinref part="U$2" gate="G$1" pin="GND(DIG)"/>
@@
 <wire x1="50.8" y1="35.56" x2="50.8" y2="56.92" width="0.1524" layer="91"/>
 <wire x1="50.8" y1="56.92" x2="54.46" y2="56.92" width="0.1524" layer="91"/>
+<label x="71.12" y="33.02" size="1.778" layer="95"/>
 </segment>
 </net>
-<net name="COLL(5V)" class="0">
+<net name="TR_PWR" class="0">
 <segment>
 <pinref part="U$1" gate="G$1" pin="5V(PWR)"/>
@@
 <wire x1="67.46" y1="56.92" x2="67.46" y2="48.26" width="0.1524" layer="91"/>
 <wire x1="67.46" y1="48.26" x2="58.42" y2="48.26" width="0.1524" layer="91"/>
+<label x="58.42" y="45.72" size="1.778" layer="95"/>
 </segment>
 </net>
-<net name="E(SIG+GND)" class="0">
+<net name="GND_A" class="0">
 <segment>
 <pinref part="U$2" gate="G$1" pin="GND(PWR)"/>
@@
 <wire x1="74.78" y1="56.92" x2="74.78" y2="40.64" width="0.1524" layer="91"/>
 <wire x1="74.78" y1="40.64" x2="58.42" y2="40.64" width="0.1524" layer="91"/>
+<label x="58.42" y="40.64" size="1.778" layer="95"/>
 </segment>
 </net>
-<net name="A(5V)" class="0">
+<net name="IR_PWR" class="0">
 <segment>
 <pinref part="1" gate="1" pin="P"/>
@@
 <wire x1="50.8" y1="66.04" x2="50.8" y2="59.92" width="0.1524" layer="91"/>
 <wire x1="50.8" y1="59.92" x2="54.46" y2="59.92" width="0.1524" layer="91"/>
+<label x="71.12" y="68.58" size="1.778" layer="95"/>
 </segment>
 </net>

Commit message: fixed
Connections:
- net GND_A: now also 4.P; no longer 3.P
- net TR_PWR: now also 3.P; no longer 4.P
Other:
- moved on the sheet: 3, 4
Changed lines of the file:
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@@
 <?xml version="1.0" encoding="utf-8"?>
 <!DOCTYPE eagle SYSTEM "eagle.dtd">
-<eagle version="8.7.0">
+<eagle version="8.7.1">
 <drawing>
 <settings>
@@
 <part name="1" library="wirepad" library_urn="urn:adsk.eagle:library:412" deviceset="2,15/1,0" device="" package3d_urn="urn:adsk.eagle:package:30831/1"/>
 <part name="2" library="wirepad" library_urn="urn:adsk.eagle:library:412" deviceset="2,15/1,0" device="" package3d_urn="urn:adsk.eagle:package:30831/1"/>
+<part name="3" library="wirepad" library_urn="urn:adsk.eagle:library:412" deviceset="2,15/1,0" device="" package3d_urn="urn:adsk.eagle:package:30831/1"/>
 <part name="4" library="wirepad" library_urn="urn:adsk.eagle:library:412" deviceset="2,15/1,0" device="" package3d_urn="urn:adsk.eagle:package:30831/1"/>
-<part name="3" library="wirepad" library_urn="urn:adsk.eagle:library:412" deviceset="2,15/1,0" device="" package3d_urn="urn:adsk.eagle:package:30831/1"/>
 </parts>
 <sheets>
@@
 <instance part="1" gate="1" x="68.58" y="71.12"/>
 <instance part="2" gate="1" x="73.66" y="30.48" rot="R180"/>
-<instance part="4" gate="1" x="55.88" y="48.26"/>
-<instance part="3" gate="1" x="55.88" y="40.64"/>
+<instance part="3" gate="1" x="55.88" y="48.26"/>
+<instance part="4" gate="1" x="55.88" y="40.64"/>
 </instances>
 <busses>
@@
 <segment>
 <pinref part="U$1" gate="G$1" pin="5V(PWR)"/>
-<pinref part="4" gate="1" pin="P"/>
+<pinref part="3" gate="1" pin="P"/>
 <wire x1="67.46" y1="56.92" x2="67.46" y2="48.26" width="0.1524" layer="91"/>
 <wire x1="67.46" y1="48.26" x2="58.42" y2="48.26" width="0.1524" layer="91"/>
@@
 <segment>
 <pinref part="U$2" gate="G$1" pin="GND(PWR)"/>
-<pinref part="3" gate="1" pin="P"/>
+<pinref part="4" gate="1" pin="P"/>
 <wire x1="74.78" y1="56.92" x2="74.78" y2="40.64" width="0.1524" layer="91"/>
 <wire x1="74.78" y1="40.64" x2="58.42" y2="40.64" width="0.1524" layer="91"/>

Commit message: updated for new part
Connections:
- net GND_A: now also 3.P; no longer 4.P
- net IR_PWR: now also 4.P; no longer 1.P
- net TR_PWR: now also 1.P; no longer 3.P
Other:
- moved on the sheet: 1, 3, 4
Changed lines of the file:
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@@
 <?xml version="1.0" encoding="utf-8"?>
 <!DOCTYPE eagle SYSTEM "eagle.dtd">
-<eagle version="8.7.1">
+<eagle version="9.0.1">
 <drawing>
 <settings>
@@
 <layers>
 <layer number="1" name="Top" color="4" fill="1" visible="no" active="no"/>
+<layer number="2" name="Route2" color="1" fill="3" visible="no" active="no"/>
+<layer number="3" name="Route3" color="4" fill="3" visible="no" active="no"/>
+<layer number="4" name="Route4" color="1" fill="4" visible="no" active="no"/>
+<layer number="5" name="Route5" color="4" fill="4" visible="no" active="no"/>
+<layer number="6" name="Route6" color="1" fill="8" visible="no" active="no"/>
+<layer number="7" name="Route7" color="4" fill="8" visible="no" active="no"/>
+<layer number="8" name="Route8" color="1" fill="2" visible="no" active="no"/>
+<layer number="9" name="Route9" color="4" fill="2" visible="no" active="no"/>
+<layer number="10" name="Route10" color="1" fill="7" visible="no" active="no"/>
+<layer number="11" name="Route11" color="4" fill="7" visible="no" active="no"/>
+<layer number="12" name="Route12" color="1" fill="5" visible="no" active="no"/>
+<layer number="13" name="Route13" color="4" fill="5" visible="no" active="no"/>
+<layer number="14" name="Route14" color="1" fill="6" visible="no" active="no"/>
+<layer number="15" name="Route15" color="4" fill="6" visible="no" active="no"/>
 <layer number="16" name="Bottom" color="1" fill="1" visible="no" active="no"/>
 <layer number="17" name="Pads" color="2" fill="1" visible="no" active="no"/>
@@
 <part name="U$1" library="ferraris_sensor_project" deviceset="CNY70" device=""/>
 <part name="U$2" library="ferraris_sensor_project" deviceset="CNY70" device=""/>
+<part name="4" library="wirepad" library_urn="urn:adsk.eagle:library:412" deviceset="2,15/1,0" device="" package3d_urn="urn:adsk.eagle:package:30831/1"/>
+<part name="2" library="wirepad" library_urn="urn:adsk.eagle:library:412" deviceset="2,15/1,0" device="" package3d_urn="urn:adsk.eagle:package:30831/1"/>
 <part name="1" library="wirepad" library_urn="urn:adsk.eagle:library:412" deviceset="2,15/1,0" device="" package3d_urn="urn:adsk.eagle:package:30831/1"/>
-<part name="2" library="wirepad" library_urn="urn:adsk.eagle:library:412" deviceset="2,15/1,0" device="" package3d_urn="urn:adsk.eagle:package:30831/1"/>
 <part name="3" library="wirepad" library_urn="urn:adsk.eagle:library:412" deviceset="2,15/1,0" device="" package3d_urn="urn:adsk.eagle:package:30831/1"/>
-<part name="4" library="wirepad" library_urn="urn:adsk.eagle:library:412" deviceset="2,15/1,0" device="" package3d_urn="urn:adsk.eagle:package:30831/1"/>
 </parts>
 <sheets>
@@
 <instance part="U$1" gate="G$1" x="60.96" y="58.42"/>
 <instance part="U$2" gate="G$1" x="81.28" y="58.42" rot="R180"/>
-<instance part="1" gate="1" x="68.58" y="71.12"/>
+<instance part="4" gate="1" x="68.58" y="71.12"/>
 <instance part="2" gate="1" x="73.66" y="30.48" rot="R180"/>
-<instance part="3" gate="1" x="55.88" y="48.26"/>
-<instance part="4" gate="1" x="55.88" y="40.64"/>
+<instance part="1" gate="1" x="55.88" y="48.26"/>
+<instance part="3" gate="1" x="55.88" y="40.64"/>
 </instances>
 <busses>
@@
 <segment>
 <pinref part="U$1" gate="G$1" pin="5V(PWR)"/>
-<pinref part="3" gate="1" pin="P"/>
+<pinref part="1" gate="1" pin="P"/>
 <wire x1="67.46" y1="56.92" x2="67.46" y2="48.26" width="0.1524" layer="91"/>
 <wire x1="67.46" y1="48.26" x2="58.42" y2="48.26" width="0.1524" layer="91"/>
@@
 <segment>
 <pinref part="U$2" gate="G$1" pin="GND(PWR)"/>
-<pinref part="4" gate="1" pin="P"/>
+<pinref part="3" gate="1" pin="P"/>
 <wire x1="74.78" y1="56.92" x2="74.78" y2="40.64" width="0.1524" layer="91"/>
 <wire x1="74.78" y1="40.64" x2="58.42" y2="40.64" width="0.1524" layer="91"/>
@@
 <net name="IR_PWR" class="0">
 <segment>
-<pinref part="1" gate="1" pin="P"/>
+<pinref part="4" gate="1" pin="P"/>
 <wire x1="71.12" y1="71.12" x2="71.12" y2="66.04" width="0.1524" layer="91"/>
 <wire x1="71.12" y1="66.04" x2="93.98" y2="66.04" width="0.1524" layer="91"/>

Commit message: fixes
Connections:
- net GND_D: now also 1.P; no longer 2.P
- net TR_PWR: now also 2.P; no longer 1.P
Other:
- moved on the sheet: 1, 2
Changed lines of the file:
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@@
 <part name="U$2" library="ferraris_sensor_project" deviceset="CNY70" device=""/>
 <part name="4" library="wirepad" library_urn="urn:adsk.eagle:library:412" deviceset="2,15/1,0" device="" package3d_urn="urn:adsk.eagle:package:30831/1"/>
+<part name="1" library="wirepad" library_urn="urn:adsk.eagle:library:412" deviceset="2,15/1,0" device="" package3d_urn="urn:adsk.eagle:package:30831/1"/>
 <part name="2" library="wirepad" library_urn="urn:adsk.eagle:library:412" deviceset="2,15/1,0" device="" package3d_urn="urn:adsk.eagle:package:30831/1"/>
-<part name="1" library="wirepad" library_urn="urn:adsk.eagle:library:412" deviceset="2,15/1,0" device="" package3d_urn="urn:adsk.eagle:package:30831/1"/>
 <part name="3" library="wirepad" library_urn="urn:adsk.eagle:library:412" deviceset="2,15/1,0" device="" package3d_urn="urn:adsk.eagle:package:30831/1"/>
 </parts>
@@
 <instance part="U$2" gate="G$1" x="81.28" y="58.42" rot="R180"/>
 <instance part="4" gate="1" x="68.58" y="71.12"/>
-<instance part="2" gate="1" x="73.66" y="30.48" rot="R180"/>
-<instance part="1" gate="1" x="55.88" y="48.26"/>
+<instance part="1" gate="1" x="73.66" y="30.48" rot="R180"/>
+<instance part="2" gate="1" x="55.88" y="48.26"/>
 <instance part="3" gate="1" x="55.88" y="40.64"/>
 </instances>
@@
 <wire x1="91.44" y1="35.56" x2="71.12" y2="35.56" width="0.1524" layer="91"/>
 <wire x1="71.12" y1="35.56" x2="50.8" y2="35.56" width="0.1524" layer="91"/>
-<pinref part="2" gate="1" pin="P"/>
+<pinref part="1" gate="1" pin="P"/>
 <wire x1="71.12" y1="30.48" x2="71.12" y2="35.56" width="0.1524" layer="91"/>
 <junction x="71.12" y="35.56"/>
@@
 <segment>
 <pinref part="U$1" gate="G$1" pin="5V(PWR)"/>
-<pinref part="1" gate="1" pin="P"/>
+<pinref part="2" gate="1" pin="P"/>
 <wire x1="67.46" y1="56.92" x2="67.46" y2="48.26" width="0.1524" layer="91"/>
 <wire x1="67.46" y1="48.26" x2="58.42" y2="48.26" width="0.1524" layer="91"/>
